Commit message: refactor: 주석 수정
glove teleop 제거. 소스·config·스크립트 삭제와 examples 빌드·plugin, bringup 의
use_glove 배선 정리. manus_ros2_msgs 조건부 빌드가 사라져 examples 가 항상 빌드된다.

examples 의 배열 크기 16 을 description.hpp 상수로 교체하고 aidin_hand2 의존 추가.

isaac 토픽 3개를 조건부로 생성하던 param 을 항상 생성하도록 바꿔 나머지 인자와 방식 통일.
기본값은 xacro 가 갖는다.

File: aidin_hand2_description/ros2_control/aidin_hand2.ros2_control.xacro (robot description, xacro)
@@ -1,14 +1,9 @@
 <?xml version="1.0"?>
-<!-- AIDIN Hand Gen2 한 손 ros2_control system — SDK(aidin_hand2) wrapper 인터페이스.
-     protocol·kinematics 는 SDK 소유. 여기는 SDK public 타입과 1:1 인 값 인터페이스만 선언한다. -->
+<!-- ros2_control system for one hand, interface declarations only -->
 <robot xmlns:xacro="http://www.ros.org/wiki/xacro">
-  <!-- Actuator 1개 — physical state만 소유한다. command는 아래 mode별 GPIO port가 소유한다.
-       state: position_cnt · velocity_rpm · current_ma (모션/센싱, hand_state_broadcaster).
-       actuator 헬스(enabled/fault)는 진단이라 아래 diagnostics gpio 로 모았다.
-       이름을 표준 position/velocity/effort 와 다르게 두는 이유: joint_state_broadcaster 가
-       count 스케일 값을 /joint_states 로 내보내지 않게 하기 위함. -->
+  <!-- =========================== Helper macro =========================== -->
+  <!-- Actuator physical state -->
   <xacro:macro name="hand_actuator" params="joint_name">
     <joint name="${joint_name}">
-      <!-- ── hand_state_broadcaster: 모션/센싱 → HandState ── -->
       <state_interface name="position_cnt"/>
       <state_interface name="velocity_rpm"/>
@@ -16,12 +11,10 @@
     </joint>
   </xacro:macro>
-  <!-- actuator 16 각각의 enabled·fault state 를 diagnostics gpio 에 방출.
-       gpio 이름(<prefix>diagnostics)이 이미 좌우를 가르므로 interface 이름엔 prefix 없이
-       actuator base 이름만 접미사로: enabled_<actuator_base>·fault_<actuator_base>. -->
+  <!-- Actuator health, suffixed with the unprefixed actuator base name -->
   <xacro:macro name="diagnostics_actuator_health" params="actuator_base">
     <state_interface name="enabled_${actuator_base}"/>
     <state_interface name="fault_${actuator_base}"/>
   </xacro:macro>
-  <!-- Joint broadcaster가 소비하는 표준 position state만 둔다. -->
+  <!-- Joint position for joint_state_broadcaster -->
   <xacro:macro name="hand_joint" params="joint_name">
     <joint name="${joint_name}">
@@ -29,5 +22,4 @@
     </joint>
   </xacro:macro>
-  <!-- state_interface 를 <prefix>idx_min..idx_max 로 방출 -->
   <xacro:macro name="state_interface_range" params="prefix idx_min idx_max">
     <state_interface name="${prefix}${idx_min}"/>
@@ -36,5 +28,5 @@
     </xacro:if>
   </xacro:macro>
-  <!-- Finger tactile — 17 cell -->
+  <!-- Finger tactile, 17 cells -->
   <xacro:macro name="finger_tactile_sensor" params="sensor_name">
     <sensor name="${sensor_name}">
@@ -42,5 +34,5 @@
     </sensor>
   </xacro:macro>
-  <!-- Palm tactile — 3 region, 58 cell -->
+  <!-- Palm tactile, 3 regions, 58 cells -->
   <xacro:macro name="palm_tactile_sensor" params="sensor_name">
     <sensor name="${sensor_name}">
@@ -50,22 +42,27 @@
     </sensor>
   </xacro:macro>
+  <!-- =========================== System macro =========================== -->
   <!--
-    한 손 ros2_control system macro. params 는 SDK OpenConfig 와 1:1 (기본값 = SDK default):
-      identity : name, prefix, hand_side
-      CAN      : can_interface
-      homing   : auto_home (on_activate 자동 homing on/off)
-      effort   : max_effort (rated current %, 0~2000)
-      control  : control_rate (RT loop Hz)
-      realtime : rt_cpu_affinity (코어 pin, -1 = 미설정)
-      reconnect: auto_reconnect (통신 두절 시 자동 재수립),
-                 auto_reconnect_timeout_ms (재수립 포기 상한, 0=무제한),
-                 auto_reconnect_home (재수립 복귀 시 run 전 homing)
-    backend 는 use_isaac > use_mock > 실 CAN 순으로 정해진다 (셋 다 같은 interface 이름 규약이라
-    controller 는 동일하게 붙는다):
-      use_isaac : Isaac Sim 과 ROS 2 토픽으로 주고받는 브리지. 실 hardware 와 같은 state 계약이라
-                  촉각·diagnostics 도 그대로 나온다.
-      use_mock  : SDK kinematics(clamp→IK→FK) mock. 촉각·diagnostics 는 내보내지 않는다.
-    isaac_* 파라미터는 use_isaac 일 때만 쓰인다. 토픽 인자가 빈 값이면 하드웨어가 topic_prefix
-    기준 기본 이름(joint_states / hand_command / tactile)을 쓴다.
+    ros2_control system macro for one hand
+    name                       ros2_control system name, and the hardware node name
+    prefix                     prepended to every joint, actuator and gpio name
+    hand_side                  "left" or "right"
+    can_interface              one CAN bus per hand, tactile included
+    auto_home                  homing on activate, otherwise the ~/home service
+    max_effort                 rated current %, 0~2000
+    control_rate               RT loop Hz
+    rt_cpu_affinity            core the RT loop is pinned to, -1 = unset
+    disabled_actuators         comma separated index list such as "0,1,2,3", empty = all on
+    auto_reconnect             reconnect after a lost link
+    auto_reconnect_timeout_ms  0 = no limit
+    auto_reconnect_home        homing before run on recovery
+    use_mock                   kinematic mock, no tactile and no diagnostics
+    use_isaac                  Isaac Sim over ROS 2 topics, taking priority over use_mock,
+                               with the same state contract as the real hardware
+    isaac_topic_prefix         the three topic names below hang off this prefix
+    isaac_joint_state_topic    Isaac to hardware, sensor_msgs/JointState
+    isaac_joint_command_topic  hardware to Isaac, sensor_msgs/JointState
+    isaac_tactile_prefix       <prefix>/<side>_<finger>_sensor, std_msgs/Float64MultiArray
+    isaac_state_timeout        seconds without a new state before the link counts as lost
   -->
   <xacro:macro name="aidin_hand2_ros2_control"
@@ -83,38 +80,15 @@
                        use_isaac:=^|false
                        isaac_topic_prefix:=^|'/isaac'
-                       isaac_joint_state_topic:=^|''
-                       isaac_joint_command_topic:=^|''
-                       isaac_tactile_prefix:=^|''
+                       isaac_joint_state_topic:=^|'joint_states'
+                       isaac_joint_command_topic:=^|'hand_command'
+                       isaac_tactile_prefix:=^|'tactile'
                        isaac_state_timeout:=^|0.1">
-    <!-- launch 에서 온 값은 'true'/'false' 문자열, dispatcher 에서 온 값은 파이썬 bool 이라
-         둘 다 받도록 정규화한다. 문자열 'false' 는 그냥 두면 참이 되어 조건이 뒤집힌다. -->
+    <!-- Takes both the 'true'/'false' string from launch and the python bool -->
     <xacro:property name="hand2_isaac" value="${str(use_isaac).lower() in ['true', '1']}"/>
     <xacro:property name="hand2_mock"
                     value="${str(use_mock).lower() in ['true', '1'] and not hand2_isaac}"/>
     <ros2_control name="${name}" type="system">
+      <!-- ====================== Hardware interface ====================== -->
       <hardware>
-        <xacro:if value="${hand2_isaac}">
-          <plugin>aidin_hand2_hardware/AidinHand2IsaacSystemInterface</plugin>
-          <param name="hand_side">${hand_side}</param>
-          <param name="max_effort">${max_effort}</param>
-          <param name="topic_prefix">${isaac_topic_prefix}</param>
-          <!-- Isaac 상태가 이 시간[s]을 넘겨 끊기면 lifecycle 이 Disconnected 로 떨어지고
-               diagnostics 의 deadline_misses 가 오른다. 0 이하면 검사하지 않는다. -->
-          <param name="state_timeout">${isaac_state_timeout}</param>
-          <xacro:if value="${isaac_joint_state_topic != ''}">
-            <param name="joint_state_topic">${isaac_joint_state_topic}</param>
-          </xacro:if>
-          <xacro:if value="${isaac_joint_command_topic != ''}">
-            <param name="joint_command_topic">${isaac_joint_command_topic}</param>
-          </xacro:if>
-          <xacro:if value="${isaac_tactile_prefix != ''}">
-            <param name="tactile_prefix">${isaac_tactile_prefix}</param>
-          </xacro:if>
-        </xacro:if>
-        <xacro:if value="${hand2_mock}">
-          <plugin>aidin_hand2_hardware/AidinHand2MockSystemInterface</plugin>
-          <param name="hand_side">${hand_side}</param>
-          <param name="max_effort">${max_effort}</param>
-        </xacro:if>
         <xacro:unless value="${hand2_isaac or hand2_mock}">
           <plugin>aidin_hand2_hardware/AidinHand2SystemInterface</plugin>
@@ -125,5 +99,4 @@
           <param name="control_rate">${control_rate}</param>
           <param name="rt_cpu_affinity">${rt_cpu_affinity}</param>
-          <!-- 미가동 actuator index (콤마 구분, 예 "0,1,2,3"). 빈 값 = 전부 가동 -->
           <param name="disabled_actuators">${disabled_actuators}</param>
           <param name="auto_reconnect">${auto_reconnect}</param>
@@ -131,6 +104,22 @@
           <param name="auto_reconnect_home">${auto_reconnect_home}</param>
         </xacro:unless>
+        <xacro:if value="${hand2_mock}">
+          <plugin>aidin_hand2_hardware/AidinHand2MockSystemInterface</plugin>
+          <param name="hand_side">${hand_side}</param>
+          <param name="max_effort">${max_effort}</param>
+        </xacro:if>
+        <xacro:if value="${hand2_isaac}">
+          <plugin>aidin_hand2_hardware/AidinHand2IsaacSystemInterface</plugin>
+          <param name="hand_side">${hand_side}</param>
+          <param name="max_effort">${max_effort}</param>
+          <param name="topic_prefix">${isaac_topic_prefix}</param>
+          <param name="state_timeout">${isaac_state_timeout}</param>
+          <param name="joint_state_topic">${isaac_joint_state_topic}</param>
+          <param name="joint_command_topic">${isaac_joint_command_topic}</param>
+          <param name="tactile_prefix">${isaac_tactile_prefix}</param>
+        </xacro:if>
       </hardware>
-      <!-- Actuator 16 = thumb 4 + long finger 3×4. 실·mock 모두 같은 physical state 계약. -->
+      <!-- =========================== Actuator =========================== -->
+      <!-- Actuator 16 = thumb 4 + long finger 3x4 -->
         <xacro:hand_actuator joint_name="${prefix}thumb_actuator0"/>
         <xacro:hand_actuator joint_name="${prefix}thumb_actuator1"/>
@@ -149,5 +138,6 @@
         <xacro:hand_actuator joint_name="${prefix}baby_actuator2"/>
         <xacro:hand_actuator joint_name="${prefix}baby_actuator3"/>
-      <!-- Joint 21 — physical position state. -->
+      <!-- ============================= Joint ============================ -->
+      <!-- Joint 21 = thumb 5 + long finger 4x4 -->
       <xacro:hand_joint joint_name="${prefix}thumb_joint0"/>
       <xacro:hand_joint joint_name="${prefix}thumb_joint1"/>
@@ -171,7 +161,8 @@
       <xacro:hand_joint joint_name="${prefix}baby_joint3"/>
       <xacro:hand_joint joint_name="${prefix}baby_joint4"/>
-      <!-- Finger/Palm tactile — mock 은 촉각 미노출(제외). Isaac 브리지는 토픽으로 받아 내보낸다. -->
+      <!-- ============================ Tactile =========================== -->
+      <!-- Finger and palm tactile, not exported by the mock -->
       <xacro:unless value="${hand2_mock}">
-        <!-- Finger tactile — 5 × 17 cell -->
+        <!-- Finger tactile, 5 x 17 cells -->
         <xacro:finger_tactile_sensor sensor_name="${prefix}thumb_sensor"/>
         <xacro:finger_tactile_sensor sensor_name="${prefix}index_sensor"/>
@@ -179,10 +170,11 @@
         <xacro:finger_tactile_sensor sensor_name="${prefix}ring_sensor"/>
         <xacro:finger_tactile_sensor sensor_name="${prefix}baby_sensor"/>
-        <!-- Palm tactile — 3 region, 58 cell -->
+        <!-- Palm tactile, 3 regions, 58 cells -->
         <xacro:palm_tactile_sensor sensor_name="${prefix}palm_sensor"/>
       </xacro:unless>
-      <!-- Homing 은 hardware 가 여는 ~/home service 로만 트리거·통지 (별도 state interface 없음) -->
-      <!-- Mode별 complete command port. 기존 4개 basic controller 중 하나만 lock과 한 port 전체를
-           claim한다. command_lock은 claim-only이며 수치값은 사용하지 않는다. -->
+      <!-- ============================ Command =========================== -->
+      <!-- Homing goes through the ~/home service, it has no state interface -->
+      <!-- One complete command port per mode, claimed whole with the lock by one controller
+           command_lock is claim-only -->
       <gpio name="${prefix}hand_control">
         <command_interface name="command_lock"/>
@@ -260,8 +252,8 @@
         <command_interface name="target_effort_pct.baby_actuator3"/>
       </gpio>
-      <!-- SDK Diagnostics 노출 — broadcaster 가 ~/hand_diagnostics 로 변환 (Stage 2).
-           hand 전역 7 필드 + actuator 16 각각의 enabled·fault. mock 은 미노출(제외).
-           Isaac 브리지는 브리지 자신이 채운 값(lifecycle·control_cycles·deadline_misses 등)을 낸다.
-           lifecycle 은 double(HandLifecycle ordinal) — broadcaster 가 이름화. -->
+      <!-- ========================== Diagnostics ========================= -->
+      <!-- Diagnostics, 7 hand-wide fields plus enabled and fault per actuator, 39 interfaces
+           Not exported by the mock
+           lifecycle and homing_state go out as ordinals, the broadcaster names them -->
       <xacro:unless value="${hand2_mock}">
       <gpio name="${prefix}diagnostics">
@@ -272,7 +264,6 @@
         <state_interface name="last_period_ms"/>
         <state_interface name="last_compute_ms"/>
-        <!-- 원점 상태 (HomingState ordinal: 0=NotRun, 1=Succeeded, 2=InProgress, 3=Failed) -->
         <state_interface name="homing_state"/>
-        <!-- per-actuator enabled·fault (actuator 16, hand_actuator 호출과 같은 순서) -->
+        <!-- Same order as the hand_actuator calls above -->
         <xacro:diagnostics_actuator_health actuator_base="thumb_actuator0"/>
         <xacro:diagnostics_actuator_health actuator_base="thumb_actuator1"/>

File: aidin_hand2_description/urdf/aidin_hand2.urdf.xacro (robot description, xacro)
@@ -1,4 +1,5 @@
 <?xml version="1.0"?>
 <robot xmlns:xacro="http://www.ros.org/wiki/xacro" name="aidin_hand2">
+  <!-- ============================= Placement ============================ -->
   <xacro:arg name="use_left_hand" default="true"/>
   <xacro:arg name="use_right_hand" default="true"/>
@@ -12,5 +13,6 @@
   <xacro:arg name="right_hand_parent" default="world"/>
   <link name="world"/>
-  <!-- 좌/우 손 link·joint·mesh 정의 -->
+  <!-- ============================= Hand URDF ============================ -->
+  <!-- Link, joint and mesh of each hand -->
   <xacro:include filename="$(find aidin_hand2_description)/urdf/aidin_hand2_left.urdf.xacro"/>
   <xacro:include filename="$(find aidin_hand2_description)/urdf/aidin_hand2_right.urdf.xacro"/>
@@ -29,37 +31,31 @@
     </xacro:aidin_hand2_right>
   </xacro:if>
-  <!-- ros2_control system 은 손마다 별도. use_left_hand / use_right_hand
-       각각에 대해 macro 호출 1번 → <ros2_control> system 1개 생성. -->
-  <xacro:include filename="$(find aidin_hand2_description)/ros2_control/aidin_hand2.ros2_control.xacro"/>
-  <!-- 손별 CAN bus. SDK 는 손당 단일 bus (tactile 포함). -->
+  <!-- ==================== Hardware interface argument =================== -->
+  <!-- Forwarded to the aidin_hand2_ros2_control macro, which documents each one -->
+  <!-- Common -->
   <xacro:arg name="left_hand_interface"   default="can0"/>
   <xacro:arg name="right_hand_interface"  default="can1"/>
-  <!-- on_activate 자동 homing on/off. 별도 트리거는 homing gpio 의 request. -->
   <xacro:arg name="auto_home"            default="true"/>
-  <!-- effort 한계 (rated current %, 0~2000). 기본값은 SDK default 와 동일. -->
   <xacro:arg name="max_effort"           default="1000"/>
-  <!-- SDK RT loop 설정. control_rate 는 loop Hz, cpu_affinity 는 격리 코어 pin 이라
-       손별 (-1 = 미설정). -->
   <xacro:arg name="control_rate"             default="500"/>
   <xacro:arg name="left_hand_cpu_affinity"   default="-1"/>
   <xacro:arg name="right_hand_cpu_affinity"  default="-1"/>
-  <!-- 미가동 actuator index (콤마 구분, 예 "0,1,2,3"). 빈 값 = 전부 가동. 손별로 지정. -->
   <xacro:arg name="left_hand_disabled_actuators"  default=""/>
   <xacro:arg name="right_hand_disabled_actuators" default=""/>
-  <!-- 통신 두절 시 SDK 자동 재수립. timeout_ms 초과면 Failed 로 종결(0=무제한),
-       home 은 재수립 복귀 시 run 전 homing 여부. 양손 공통 정책. -->
   <xacro:arg name="auto_reconnect"            default="false"/>
   <xacro:arg name="auto_reconnect_timeout_ms" default="0"/>
   <xacro:arg name="auto_reconnect_home"       default="false"/>
-  <!-- true 면 실 CAN 대신 kinematics mock(clamp→IK→FK) hardware 사용 -->
+  <!-- Mock only -->
   <xacro:arg name="use_mock" default="false"/>
-  <!-- true 면 Isaac Sim 브리지 hardware 사용 (use_mock 보다 우선). 토픽은 topic_prefix 기준
-       기본 이름(joint_states / hand_command / tactile)을 쓰고, 아래 인자로 개별 지정한다. -->
+  <!-- Isaac only -->
   <xacro:arg name="use_isaac" default="false"/>
   <xacro:arg name="isaac_topic_prefix"       default="/isaac"/>
-  <xacro:arg name="isaac_joint_state_topic"  default=""/>
-  <xacro:arg name="isaac_joint_command_topic" default=""/>
-  <xacro:arg name="isaac_tactile_prefix"     default=""/>
+  <xacro:arg name="isaac_joint_state_topic"  default="joint_states"/>
+  <xacro:arg name="isaac_joint_command_topic" default="hand_command"/>
+  <xacro:arg name="isaac_tactile_prefix"     default="tactile"/>
   <xacro:arg name="isaac_state_timeout"      default="0.1"/>
+  <!-- ======================== ros2_control system ======================= -->
+  <!-- One ros2_control system per hand -->
+  <xacro:include filename="$(find aidin_hand2_description)/ros2_control/aidin_hand2.ros2_control.xacro"/>
   <xacro:if value="$(arg use_left_hand)">
     <xacro:aidin_hand2_ros2_control

File: aidin_hand2_description/urdf/aidin_hand2_left.urdf.xacro (robot description, xacro)
@@ -5,10 +5,10 @@
   XZ plane (M = diag(1,-1,1), i.e. Y -> -Y).  Per-element rule:
     - link/joint origin xyz : negate Y
-    - link/joint origin rpy : R' = M R M  (재계산)
-    - inertia tensor        : ixy, iyz 부호 반전 (ixx/iyy/izz/ixz 불변)
+    - link/joint origin rpy : R' = M R M  (recomputed)
+    - inertia tensor        : ixy, iyz sign flipped (ixx/iyy/izz/ixz unchanged)
     - joint axis            : a' = -M a
-    - mass / limit / effort / velocity : 불변 (right와 동일)
+    - mass / limit / effort / velocity : unchanged
     - palm mesh             : body_right.STL -> body_left.STL
-    - 손가락 mesh           : 좌우 공용 STL 재사용 + link-local Y scale 로 mirror
+    - finger mesh           : the shared STL, mirrored by a link-local Y scale
 -->
 <robot xmlns:xacro="http://www.ros.org/wiki/xacro">
@@ -21,5 +21,5 @@
       <xacro:insert_block name="origin"/>
     </joint>
-    <!-- ================================ base link ================================ -->
+    <!-- ============================ Base link =========================== -->
     <link name="${prefix}hand_base_link">
       <inertial>
@@ -47,5 +47,5 @@
       </collision>
     </link>
-    <!-- ================================ thumb  ================================ -->
+    <!-- ============================== Thumb ============================= -->
     <link name="${prefix}thumb_link0">
       <inertial>
@@ -192,5 +192,5 @@
       <child link="${prefix}thumb_link2"/>
       <axis xyz="0 1 0"/>
-      <limit lower="-0.787143" upper="0.787143" effort="1.2" velocity="1.57"/>  <!-- ±45.1° — joint_clamp.cpp 의 thumb plateau (실측) -->
+      <limit lower="-0.787143" upper="0.787143" effort="1.2" velocity="1.57"/>  <!-- ±45.1°, the thumb plateau in joint_clamp.cpp -->
     </joint>
     <joint name="${prefix}thumb_joint3" type="revolute">
@@ -206,7 +206,7 @@
       <child link="${prefix}thumb_link4"/>
       <axis xyz="0 1 0"/>
-      <limit lower="0" upper="1.500202" effort="1.2" velocity="1.57"/>  <!-- passive: q3 70° 에서 유도 (IP four-bar) -->
-    </joint>
-    <!-- ================================ index finger ================================ -->
+      <limit lower="0" upper="1.500202" effort="1.2" velocity="1.57"/>  <!-- Passive, derived from joint3 at 70°, IP four-bar -->
+    </joint>
+    <!-- ========================== Index finger ========================== -->
     <link name="${prefix}index_link1">
       <inertial>
@@ -335,7 +335,7 @@
       <child link="${prefix}index_link4"/>
       <axis xyz="0 1 0"/>
-      <limit lower="0" upper="1.739111" effort="1.2" velocity="1.57"/>  <!-- passive: q3 90° 에서 유도 (four-bar) -->
-    </joint>
-    <!-- ================================ middle finger ================================ -->
+      <limit lower="0" upper="1.739111" effort="1.2" velocity="1.57"/>  <!-- Passive, derived from joint3 at 90°, four-bar -->
+    </joint>
+    <!-- ========================== Middle finger ========================= -->
     <link name="${prefix}middle_link1">
       <inertial>
@@ -464,7 +464,7 @@
       <child link="${prefix}middle_link4"/>
       <axis xyz="0 1 0"/>
-      <limit lower="0" upper="1.739111" effort="1.2" velocity="1.57"/>  <!-- passive: q3 90° 에서 유도 (four-bar) -->
-    </joint>
-    <!-- ================================ ring finger ================================ -->
+      <limit lower="0" upper="1.739111" effort="1.2" velocity="1.57"/>  <!-- Passive, derived from joint3 at 90°, four-bar -->
+    </joint>
+    <!-- =========================== Ring finger ========================== -->
     <link name="${prefix}ring_link1">
       <inertial>
@@ -593,7 +593,7 @@
       <child link="${prefix}ring_link4"/>
       <axis xyz="0 1 0"/>
-      <limit lower="0" upper="1.739111" effort="1.2" velocity="1.57"/>  <!-- passive: q3 90° 에서 유도 (four-bar) -->
-    </joint>
-    <!-- ================================ baby finger ================================ -->
+      <limit lower="0" upper="1.739111" effort="1.2" velocity="1.57"/>  <!-- Passive, derived from joint3 at 90°, four-bar -->
+    </joint>
+    <!-- =========================== Baby finger ========================== -->
     <link name="${prefix}baby_link1">
       <inertial>
@@ -722,5 +722,5 @@
       <child link="${prefix}baby_link4"/>
       <axis xyz="0 1 0"/>
-      <limit lower="0" upper="1.739111" effort="1.2" velocity="1.57"/>  <!-- passive: q3 90° 에서 유도 (four-bar) -->
+      <limit lower="0" upper="1.739111" effort="1.2" velocity="1.57"/>  <!-- Passive, derived from joint3 at 90°, four-bar -->
     </joint>
   </xacro:macro>
