Commit message: refactor: 주석 수정
glove teleop 제거. 소스·config·스크립트 삭제와 examples 빌드·plugin, bringup 의
use_glove 배선 정리. manus_ros2_msgs 조건부 빌드가 사라져 examples 가 항상 빌드된다.

examples 의 배열 크기 16 을 description.hpp 상수로 교체하고 aidin_hand2 의존 추가.

isaac 토픽 3개를 조건부로 생성하던 param 을 항상 생성하도록 바꿔 나머지 인자와 방식 통일.
기본값은 xacro 가 갖는다.

File: aidin_hand2_description/urdf/aidin_hand2_right.urdf.xacro (robot description, xacro)
@@ -14,5 +14,5 @@
       <xacro:insert_block name="origin"/>
     </joint>
-    <!-- ================================ base link ================================ -->
+    <!-- ============================ Base link =========================== -->
     <link name="${prefix}hand_base_link">
       <inertial>
@@ -40,5 +40,5 @@
       </collision>
     </link>
-    <!-- ================================ thumb  ================================ -->
+    <!-- ============================== Thumb ============================= -->
     <link name="${prefix}thumb_link0">
       <inertial>
@@ -185,5 +185,5 @@
       <child link="${prefix}thumb_link2"/>
       <axis xyz="0 1 0"/>
-      <limit lower="-0.787143" upper="0.787143" effort="1.2" velocity="1.57"/>  <!-- ±45.1° — joint_clamp.cpp 의 thumb plateau (실측) -->
+      <limit lower="-0.787143" upper="0.787143" effort="1.2" velocity="1.57"/>  <!-- ±45.1°, the thumb plateau in joint_clamp.cpp -->
     </joint>
     <joint name="${prefix}thumb_joint3" type="revolute">
@@ -199,7 +199,7 @@
       <child link="${prefix}thumb_link4"/>
       <axis xyz="0 1 0"/>
-      <limit lower="0" upper="1.500202" effort="1.2" velocity="1.57"/>  <!-- passive: q3 70° 에서 유도 (IP four-bar) -->
-    </joint>
-    <!-- ================================ index finger ================================ -->
+      <limit lower="0" upper="1.500202" effort="1.2" velocity="1.57"/>  <!-- Passive, derived from joint3 at 70°, IP four-bar -->
+    </joint>
+    <!-- ========================== Index finger ========================== -->
     <link name="${prefix}index_link1">
       <inertial>
@@ -328,7 +328,7 @@
       <child link="${prefix}index_link4"/>
       <axis xyz="0 1 0"/>
-      <limit lower="0" upper="1.739111" effort="1.2" velocity="1.57"/>  <!-- passive: q3 90° 에서 유도 (four-bar) -->
-    </joint>
-    <!-- ================================ middle finger ================================ -->
+      <limit lower="0" upper="1.739111" effort="1.2" velocity="1.57"/>  <!-- Passive, derived from joint3 at 90°, four-bar -->
+    </joint>
+    <!-- ========================== Middle finger ========================= -->
     <link name="${prefix}middle_link1">
       <inertial>
@@ -457,7 +457,7 @@
       <child link="${prefix}middle_link4"/>
       <axis xyz="0 1 0"/>
-      <limit lower="0" upper="1.739111" effort="1.2" velocity="1.57"/>  <!-- passive: q3 90° 에서 유도 (four-bar) -->
-    </joint>
-    <!-- ================================ ring finger ================================ -->
+      <limit lower="0" upper="1.739111" effort="1.2" velocity="1.57"/>  <!-- Passive, derived from joint3 at 90°, four-bar -->
+    </joint>
+    <!-- =========================== Ring finger ========================== -->
     <link name="${prefix}ring_link1">
       <inertial>
@@ -586,7 +586,7 @@
       <child link="${prefix}ring_link4"/>
       <axis xyz="0 1 0"/>
-      <limit lower="0" upper="1.739111" effort="1.2" velocity="1.57"/>  <!-- passive: q3 90° 에서 유도 (four-bar) -->
-    </joint>
-    <!-- ================================ baby finger ================================ -->
+      <limit lower="0" upper="1.739111" effort="1.2" velocity="1.57"/>  <!-- Passive, derived from joint3 at 90°, four-bar -->
+    </joint>
+    <!-- =========================== Baby finger ========================== -->
     <link name="${prefix}baby_link1">
       <inertial>
@@ -715,5 +715,5 @@
       <child link="${prefix}baby_link4"/>
       <axis xyz="0 1 0"/>
-      <limit lower="0" upper="1.739111" effort="1.2" velocity="1.57"/>  <!-- passive: q3 90° 에서 유도 (four-bar) -->
+      <limit lower="0" upper="1.739111" effort="1.2" velocity="1.57"/>  <!-- Passive, derived from joint3 at 90°, four-bar -->
     </joint>
   </xacro:macro>

Commit message: refactor: Remove the Isaac Sim backend
The Isaac plugin, its launch file, controller config and the
use_isaac / isaac_* macro arguments are gone. The robot hand and the
mock remain, selected by use_mock. The backend is not maintained
against the current SDK and will return once the wrapper framework
is stable. The CHANGELOG carries the Breaking entry.

File: aidin_hand2_description/ros2_control/aidin_hand2.ros2_control.xacro (robot description, xacro)
@@ -58,11 +58,4 @@
     auto_reconnect_home        homing before run on recovery
     use_mock                   kinematic mock, no tactile and no diagnostics
-    use_isaac                  Isaac Sim over ROS 2 topics, taking priority over use_mock,
-                               with the same state contract as the real hardware
-    isaac_topic_prefix         the three topic names below hang off this prefix
-    isaac_joint_state_topic    Isaac to hardware, sensor_msgs/JointState
-    isaac_joint_command_topic  hardware to Isaac, sensor_msgs/JointState
-    isaac_tactile_prefix       <prefix>/<side>_<finger>_sensor, std_msgs/Float64MultiArray
-    isaac_state_timeout        seconds without a new state before the link counts as lost
   -->
   <xacro:macro name="aidin_hand2_ros2_control"
@@ -77,19 +70,11 @@
                        auto_reconnect_timeout_ms:=^|0
                        auto_reconnect_home:=^|false
-                       use_mock:=^|false
-                       use_isaac:=^|false
-                       isaac_topic_prefix:=^|'/isaac'
-                       isaac_joint_state_topic:=^|'joint_states'
-                       isaac_joint_command_topic:=^|'hand_command'
-                       isaac_tactile_prefix:=^|'tactile'
-                       isaac_state_timeout:=^|0.1">
+                       use_mock:=^|false">
     <!-- Takes both the 'true'/'false' string from launch and the python bool -->
-    <xacro:property name="hand2_isaac" value="${str(use_isaac).lower() in ['true', '1']}"/>
-    <xacro:property name="hand2_mock"
-                    value="${str(use_mock).lower() in ['true', '1'] and not hand2_isaac}"/>
+    <xacro:property name="hand2_mock" value="${str(use_mock).lower() in ['true', '1']}"/>
     <ros2_control name="${name}" type="system">
       <!-- ====================== Hardware interface ====================== -->
       <hardware>
-        <xacro:unless value="${hand2_isaac or hand2_mock}">
+        <xacro:unless value="${hand2_mock}">
           <plugin>aidin_hand2_hardware/AidinHand2SystemInterface</plugin>
           <param name="hand_side">${hand_side}</param>
@@ -108,14 +93,4 @@
           <param name="hand_side">${hand_side}</param>
           <param name="max_effort">${max_effort}</param>
-        </xacro:if>
-        <xacro:if value="${hand2_isaac}">
-          <plugin>aidin_hand2_hardware/AidinHand2IsaacSystemInterface</plugin>
-          <param name="hand_side">${hand_side}</param>
-          <param name="max_effort">${max_effort}</param>
-          <param name="topic_prefix">${isaac_topic_prefix}</param>
-          <param name="state_timeout">${isaac_state_timeout}</param>
-          <param name="joint_state_topic">${isaac_joint_state_topic}</param>
-          <param name="joint_command_topic">${isaac_joint_command_topic}</param>
-          <param name="tactile_prefix">${isaac_tactile_prefix}</param>
         </xacro:if>
       </hardware>

File: aidin_hand2_description/urdf/aidin_hand2.urdf.xacro (robot description, xacro)
@@ -48,11 +48,4 @@
   <!-- Mock only -->
   <xacro:arg name="use_mock" default="false"/>
-  <!-- Isaac only -->
-  <xacro:arg name="use_isaac" default="false"/>
-  <xacro:arg name="isaac_topic_prefix"       default="/isaac"/>
-  <xacro:arg name="isaac_joint_state_topic"  default="joint_states"/>
-  <xacro:arg name="isaac_joint_command_topic" default="hand_command"/>
-  <xacro:arg name="isaac_tactile_prefix"     default="tactile"/>
-  <xacro:arg name="isaac_state_timeout"      default="0.1"/>
   <!-- ======================== ros2_control system ======================= -->
   <!-- One ros2_control system per hand -->
@@ -72,11 +65,5 @@
       auto_reconnect_timeout_ms="$(arg auto_reconnect_timeout_ms)"
       auto_reconnect_home="$(arg auto_reconnect_home)"
-      use_mock="$(arg use_mock)"
-      use_isaac="$(arg use_isaac)"
-      isaac_topic_prefix="$(arg isaac_topic_prefix)"
-      isaac_joint_state_topic="$(arg isaac_joint_state_topic)"
-      isaac_joint_command_topic="$(arg isaac_joint_command_topic)"
-      isaac_tactile_prefix="$(arg isaac_tactile_prefix)"
-      isaac_state_timeout="$(arg isaac_state_timeout)"/>
+      use_mock="$(arg use_mock)"/>
   </xacro:if>
   <xacro:if value="$(arg use_right_hand)">
@@ -94,11 +81,5 @@
       auto_reconnect_timeout_ms="$(arg auto_reconnect_timeout_ms)"
       auto_reconnect_home="$(arg auto_reconnect_home)"
-      use_mock="$(arg use_mock)"
-      use_isaac="$(arg use_isaac)"
-      isaac_topic_prefix="$(arg isaac_topic_prefix)"
-      isaac_joint_state_topic="$(arg isaac_joint_state_topic)"
-      isaac_joint_command_topic="$(arg isaac_joint_command_topic)"
-      isaac_tactile_prefix="$(arg isaac_tactile_prefix)"
-      isaac_state_timeout="$(arg isaac_state_timeout)"/>
+      use_mock="$(arg use_mock)"/>
   </xacro:if>
 </robot>
