Commit message: feat: Restore the Isaac Sim backend on Jazzy
Reverts 7d2938d so aidin_rby1_description can run the Gen2 hand against Isaac Sim
with hardware_mode:=isaac, and ports the restored pieces to Jazzy:
- Isaac hardware on_init takes HardwareComponentInterfaceParams
- The Isaac launch reads robot_description from the topic

Co-Authored-By: Claude Opus 5.5 <noreply@anthropic.com>

File: aidin_hand2_description/ros2_control/aidin_hand2.ros2_control.xacro (robot description, xacro)
@@ -58,4 +58,11 @@
     auto_reconnect_home        homing before run on recovery
     use_mock                   kinematic mock, no tactile and no diagnostics
+    use_isaac                  Isaac Sim over ROS 2 topics, taking priority over use_mock,
+                               with the same state contract as the real hardware
+    isaac_topic_prefix         the three topic names below hang off this prefix
+    isaac_joint_state_topic    Isaac to hardware, sensor_msgs/JointState
+    isaac_joint_command_topic  hardware to Isaac, sensor_msgs/JointState
+    isaac_tactile_prefix       <prefix>/<side>_<finger>_sensor, std_msgs/Float64MultiArray
+    isaac_state_timeout        seconds without a new state before the link counts as lost
   -->
   <xacro:macro name="aidin_hand2_ros2_control"
@@ -70,11 +77,19 @@
                        auto_reconnect_timeout_ms:=^|0
                        auto_reconnect_home:=^|false
-                       use_mock:=^|false">
+                       use_mock:=^|false
+                       use_isaac:=^|false
+                       isaac_topic_prefix:=^|'/isaac'
+                       isaac_joint_state_topic:=^|'joint_states'
+                       isaac_joint_command_topic:=^|'hand_command'
+                       isaac_tactile_prefix:=^|'tactile'
+                       isaac_state_timeout:=^|0.1">
     <!-- Takes both the 'true'/'false' string from launch and the python bool -->
-    <xacro:property name="hand2_mock" value="${str(use_mock).lower() in ['true', '1']}"/>
+    <xacro:property name="hand2_isaac" value="${str(use_isaac).lower() in ['true', '1']}"/>
+    <xacro:property name="hand2_mock"
+                    value="${str(use_mock).lower() in ['true', '1'] and not hand2_isaac}"/>
     <ros2_control name="${name}" type="system">
       <!-- ====================== Hardware interface ====================== -->
       <hardware>
-        <xacro:unless value="${hand2_mock}">
+        <xacro:unless value="${hand2_isaac or hand2_mock}">
           <plugin>aidin_hand2_hardware/AidinHand2SystemInterface</plugin>
           <param name="hand_side">${hand_side}</param>
@@ -93,4 +108,14 @@
           <param name="hand_side">${hand_side}</param>
           <param name="max_effort">${max_effort}</param>
+        </xacro:if>
+        <xacro:if value="${hand2_isaac}">
+          <plugin>aidin_hand2_hardware/AidinHand2IsaacSystemInterface</plugin>
+          <param name="hand_side">${hand_side}</param>
+          <param name="max_effort">${max_effort}</param>
+          <param name="topic_prefix">${isaac_topic_prefix}</param>
+          <param name="state_timeout">${isaac_state_timeout}</param>
+          <param name="joint_state_topic">${isaac_joint_state_topic}</param>
+          <param name="joint_command_topic">${isaac_joint_command_topic}</param>
+          <param name="tactile_prefix">${isaac_tactile_prefix}</param>
         </xacro:if>
       </hardware>

File: aidin_hand2_description/xacro/aidin_hand2.urdf.xacro (robot description, xacro)
@@ -48,4 +48,11 @@
   <!-- Mock only -->
   <xacro:arg name="use_mock" default="false"/>
+  <!-- Isaac only -->
+  <xacro:arg name="use_isaac" default="false"/>
+  <xacro:arg name="isaac_topic_prefix"       default="/isaac"/>
+  <xacro:arg name="isaac_joint_state_topic"  default="joint_states"/>
+  <xacro:arg name="isaac_joint_command_topic" default="hand_command"/>
+  <xacro:arg name="isaac_tactile_prefix"     default="tactile"/>
+  <xacro:arg name="isaac_state_timeout"      default="0.1"/>
   <!-- ======================== ros2_control system ======================= -->
   <!-- One ros2_control system per hand -->
@@ -65,5 +72,11 @@
       auto_reconnect_timeout_ms="$(arg auto_reconnect_timeout_ms)"
       auto_reconnect_home="$(arg auto_reconnect_home)"
-      use_mock="$(arg use_mock)"/>
+      use_mock="$(arg use_mock)"
+      use_isaac="$(arg use_isaac)"
+      isaac_topic_prefix="$(arg isaac_topic_prefix)"
+      isaac_joint_state_topic="$(arg isaac_joint_state_topic)"
+      isaac_joint_command_topic="$(arg isaac_joint_command_topic)"
+      isaac_tactile_prefix="$(arg isaac_tactile_prefix)"
+      isaac_state_timeout="$(arg isaac_state_timeout)"/>
   </xacro:if>
   <xacro:if value="$(arg use_right_hand)">
@@ -81,5 +94,11 @@
       auto_reconnect_timeout_ms="$(arg auto_reconnect_timeout_ms)"
       auto_reconnect_home="$(arg auto_reconnect_home)"
-      use_mock="$(arg use_mock)"/>
+      use_mock="$(arg use_mock)"
+      use_isaac="$(arg use_isaac)"
+      isaac_topic_prefix="$(arg isaac_topic_prefix)"
+      isaac_joint_state_topic="$(arg isaac_joint_state_topic)"
+      isaac_joint_command_topic="$(arg isaac_joint_command_topic)"
+      isaac_tactile_prefix="$(arg isaac_tactile_prefix)"
+      isaac_state_timeout="$(arg isaac_state_timeout)"/>
   </xacro:if>
 </robot>
