Commit message: fix: URDF joint limit 을 clamp 실측값으로 정정
joint_clamp.cpp 의 측정 경계와 어긋나 있던 active 16 을 맞추고, passive
q4 5 개는 q3 한계에서 four-bar 로 유도.

File: aidin_hand2_description/urdf/aidin_hand2_left.urdf.xacro (robot description, xacro)
@@ -178,5 +178,5 @@
       <child link="${prefix}thumb_link0"/>
       <axis xyz="0 1 0"/>
-      <limit lower="0" upper="1.9461" effort="1.2" velocity="1.57"/>
+      <limit lower="0" upper="1.919862" effort="1.2" velocity="1.57"/>
     </joint>
     <joint name="${prefix}thumb_joint1" type="revolute">
@@ -185,5 +185,5 @@
       <child link="${prefix}thumb_link1"/>
       <axis xyz="0 1 0"/>
-      <limit lower="0" upper="0.7767" effort="1.2" velocity="1.57"/>
+      <limit lower="0" upper="1.330464" effort="1.2" velocity="1.57"/>
     </joint>
     <joint name="${prefix}thumb_joint2" type="revolute">
@@ -192,5 +192,5 @@
       <child link="${prefix}thumb_link2"/>
       <axis xyz="0 1 0"/>
-      <limit lower="-0.5236" upper="0.5236" effort="1.2" velocity="1.57"/>  <!-- ±30° (2026-07-28 실측) -->
+      <limit lower="-0.787143" upper="0.787143" effort="1.2" velocity="1.57"/>  <!-- ±45.1° — joint_clamp.cpp 의 thumb plateau (실측) -->
     </joint>
     <joint name="${prefix}thumb_joint3" type="revolute">
@@ -199,5 +199,5 @@
       <child link="${prefix}thumb_link3"/>
       <axis xyz="0 1 0"/>
-      <limit lower="0" upper="1.309" effort="1.2" velocity="1.57"/>
+      <limit lower="0" upper="1.22173" effort="1.2" velocity="1.57"/>
     </joint>
     <joint name="${prefix}thumb_joint4" type="revolute">
@@ -206,5 +206,5 @@
       <child link="${prefix}thumb_link4"/>
       <axis xyz="0 1 0"/>
-      <limit lower="0" upper="1.6581" effort="1.2" velocity="1.57"/>
+      <limit lower="0" upper="1.500202" effort="1.2" velocity="1.57"/>  <!-- passive: q3 70° 에서 유도 (IP four-bar) -->
     </joint>
     <!-- ================================ index finger ================================ -->
@@ -314,5 +314,5 @@
       <child link="${prefix}index_link1"/>
       <axis xyz="0 1 0"/>
-      <limit lower="-0.5236" upper="0.5236" effort="1.2" velocity="1.57"/>
+      <limit lower="-0.479966" upper="0.479966" effort="1.2" velocity="1.57"/>
     </joint>
     <joint name="${prefix}index_joint2" type="revolute">
@@ -321,5 +321,5 @@
       <child link="${prefix}index_link2"/>
       <axis xyz="0 1 0"/>
-      <limit lower="0" upper="1.6581" effort="1.2" velocity="1.57"/>
+      <limit lower="0" upper="1.666091" effort="1.2" velocity="1.57"/>
     </joint>
     <joint name="${prefix}index_joint3" type="revolute">
@@ -328,5 +328,5 @@
       <child link="${prefix}index_link3"/>
       <axis xyz="0 1 0"/>
-      <limit lower="0" upper="1.5533" effort="1.2" velocity="1.57"/>
+      <limit lower="0" upper="1.570796" effort="1.2" velocity="1.57"/>
     </joint>
     <joint name="${prefix}index_joint4" type="revolute">
@@ -335,5 +335,5 @@
       <child link="${prefix}index_link4"/>
       <axis xyz="0 1 0"/>
-      <limit lower="0" upper="1.6319" effort="1.2" velocity="1.57"/>
+      <limit lower="0" upper="1.739111" effort="1.2" velocity="1.57"/>  <!-- passive: q3 90° 에서 유도 (four-bar) -->
     </joint>
     <!-- ================================ middle finger ================================ -->
@@ -443,5 +443,5 @@
       <child link="${prefix}middle_link1"/>
       <axis xyz="0 1 0"/>
-      <limit lower="-0.5236" upper="0.5236" effort="1.2" velocity="1.57"/>
+      <limit lower="-0.479966" upper="0.479966" effort="1.2" velocity="1.57"/>
     </joint>
     <joint name="${prefix}middle_joint2" type="revolute">
@@ -450,5 +450,5 @@
       <child link="${prefix}middle_link2"/>
       <axis xyz="0 1 0"/>
-      <limit lower="0" upper="1.6581" effort="1.2" velocity="1.57"/>
+      <limit lower="0" upper="1.666091" effort="1.2" velocity="1.57"/>
     </joint>
     <joint name="${prefix}middle_joint3" type="revolute">
@@ -457,5 +457,5 @@
       <child link="${prefix}middle_link3"/>
       <axis xyz="0 1 0"/>
-      <limit lower="0" upper="1.5533" effort="1.2" velocity="1.57"/>
+      <limit lower="0" upper="1.570796" effort="1.2" velocity="1.57"/>
     </joint>
     <joint name="${prefix}middle_joint4" type="revolute">
@@ -464,5 +464,5 @@
       <child link="${prefix}middle_link4"/>
       <axis xyz="0 1 0"/>
-      <limit lower="0" upper="1.6319" effort="1.2" velocity="1.57"/>
+      <limit lower="0" upper="1.739111" effort="1.2" velocity="1.57"/>  <!-- passive: q3 90° 에서 유도 (four-bar) -->
     </joint>
     <!-- ================================ ring finger ================================ -->
@@ -572,5 +572,5 @@
       <child link="${prefix}ring_link1"/>
       <axis xyz="0 1 0"/>
-      <limit lower="-0.5236" upper="0.5236" effort="1.2" velocity="1.57"/>
+      <limit lower="-0.479966" upper="0.479966" effort="1.2" velocity="1.57"/>
     </joint>
     <joint name="${prefix}ring_joint2" type="revolute">
@@ -579,5 +579,5 @@
       <child link="${prefix}ring_link2"/>
       <axis xyz="0 1 0"/>
-      <limit lower="0" upper="1.6581" effort="1.2" velocity="1.57"/>
+      <limit lower="0" upper="1.666091" effort="1.2" velocity="1.57"/>
     </joint>
     <joint name="${prefix}ring_joint3" type="revolute">
@@ -586,5 +586,5 @@
       <child link="${prefix}ring_link3"/>
       <axis xyz="0 1 0"/>
-      <limit lower="0" upper="1.5533" effort="1.2" velocity="1.57"/>
+      <limit lower="0" upper="1.570796" effort="1.2" velocity="1.57"/>
     </joint>
     <joint name="${prefix}ring_joint4" type="revolute">
@@ -593,5 +593,5 @@
       <child link="${prefix}ring_link4"/>
       <axis xyz="0 1 0"/>
-      <limit lower="0" upper="1.6319" effort="1.2" velocity="1.57"/>
+      <limit lower="0" upper="1.739111" effort="1.2" velocity="1.57"/>  <!-- passive: q3 90° 에서 유도 (four-bar) -->
     </joint>
     <!-- ================================ baby finger ================================ -->
@@ -701,5 +701,5 @@
       <child link="${prefix}baby_link1"/>
       <axis xyz="0 1 0"/>
-      <limit lower="-0.5236" upper="0.5236" effort="1.2" velocity="1.57"/>
+      <limit lower="-0.479966" upper="0.479966" effort="1.2" velocity="1.57"/>
     </joint>
     <joint name="${prefix}baby_joint2" type="revolute">
@@ -708,5 +708,5 @@
       <child link="${prefix}baby_link2"/>
       <axis xyz="0 1 0"/>
-      <limit lower="0" upper="1.6581" effort="1.2" velocity="1.57"/>
+      <limit lower="0" upper="1.666091" effort="1.2" velocity="1.57"/>
     </joint>
     <joint name="${prefix}baby_joint3" type="revolute">
@@ -715,5 +715,5 @@
       <child link="${prefix}baby_link3"/>
       <axis xyz="0 1 0"/>
-      <limit lower="0" upper="1.5533" effort="1.2" velocity="1.57"/>
+      <limit lower="0" upper="1.570796" effort="1.2" velocity="1.57"/>
     </joint>
     <joint name="${prefix}baby_joint4" type="revolute">
@@ -722,5 +722,5 @@
       <child link="${prefix}baby_link4"/>
       <axis xyz="0 1 0"/>
-      <limit lower="0" upper="1.6319" effort="1.2" velocity="1.57"/>
+      <limit lower="0" upper="1.739111" effort="1.2" velocity="1.57"/>  <!-- passive: q3 90° 에서 유도 (four-bar) -->
     </joint>
   </xacro:macro>

File: aidin_hand2_description/urdf/aidin_hand2_right.urdf.xacro (robot description, xacro)
@@ -171,5 +171,5 @@
       <child link="${prefix}thumb_link0"/>
       <axis xyz="0 1 0"/>
-      <limit lower="0" upper="1.9461" effort="1.2" velocity="1.57"/>
+      <limit lower="0" upper="1.919862" effort="1.2" velocity="1.57"/>
     </joint>
     <joint name="${prefix}thumb_joint1" type="revolute">
@@ -178,5 +178,5 @@
       <child link="${prefix}thumb_link1"/>
       <axis xyz="0 1 0"/>
-      <limit lower="0" upper="1.0518" effort="1.2" velocity="1.57"/>
+      <limit lower="0" upper="1.330464" effort="1.2" velocity="1.57"/>
     </joint>
     <joint name="${prefix}thumb_joint2" type="revolute">
@@ -185,5 +185,5 @@
       <child link="${prefix}thumb_link2"/>
       <axis xyz="0 1 0"/>
-      <limit lower="-0.5236" upper="0.5236" effort="1.2" velocity="1.57"/>  <!-- ±30° (2026-07-28 실측) -->
+      <limit lower="-0.787143" upper="0.787143" effort="1.2" velocity="1.57"/>  <!-- ±45.1° — joint_clamp.cpp 의 thumb plateau (실측) -->
     </joint>
     <joint name="${prefix}thumb_joint3" type="revolute">
@@ -192,5 +192,5 @@
       <child link="${prefix}thumb_link3"/>
       <axis xyz="0 1 0"/>
-      <limit lower="0" upper="1.231" effort="1.2" velocity="1.57"/>
+      <limit lower="0" upper="1.22173" effort="1.2" velocity="1.57"/>
     </joint>
     <joint name="${prefix}thumb_joint4" type="revolute">
@@ -199,5 +199,5 @@
       <child link="${prefix}thumb_link4"/>
       <axis xyz="0 1 0"/>
-      <limit lower="0" upper="1.6581" effort="1.2" velocity="1.57"/>
+      <limit lower="0" upper="1.500202" effort="1.2" velocity="1.57"/>  <!-- passive: q3 70° 에서 유도 (IP four-bar) -->
     </joint>
     <!-- ================================ index finger ================================ -->
@@ -307,5 +307,5 @@
       <child link="${prefix}index_link1"/>
       <axis xyz="0 1 0"/>
-      <limit lower="-0.5236" upper="0.5236" effort="1.2" velocity="1.57"/>
+      <limit lower="-0.479966" upper="0.479966" effort="1.2" velocity="1.57"/>
     </joint>
     <joint name="${prefix}index_joint2" type="revolute">
@@ -314,5 +314,5 @@
       <child link="${prefix}index_link2"/>
       <axis xyz="0 1 0"/>
-      <limit lower="0" upper="1.6581" effort="1.2" velocity="1.57"/>
+      <limit lower="0" upper="1.666091" effort="1.2" velocity="1.57"/>
     </joint>
     <joint name="${prefix}index_joint3" type="revolute">
@@ -321,5 +321,5 @@
       <child link="${prefix}index_link3"/>
       <axis xyz="0 1 0"/>
-      <limit lower="0" upper="1.5533" effort="1.2" velocity="1.57"/>
+      <limit lower="0" upper="1.570796" effort="1.2" velocity="1.57"/>
     </joint>
     <joint name="${prefix}index_joint4" type="revolute">
@@ -328,5 +328,5 @@
       <child link="${prefix}index_link4"/>
       <axis xyz="0 1 0"/>
-      <limit lower="0" upper="1.6319" effort="1.2" velocity="1.57"/>
+      <limit lower="0" upper="1.739111" effort="1.2" velocity="1.57"/>  <!-- passive: q3 90° 에서 유도 (four-bar) -->
     </joint>
     <!-- ================================ middle finger ================================ -->
@@ -436,5 +436,5 @@
       <child link="${prefix}middle_link1"/>
       <axis xyz="0 1 0"/>
-      <limit lower="-0.5236" upper="0.5236" effort="1.2" velocity="1.57"/>
+      <limit lower="-0.479966" upper="0.479966" effort="1.2" velocity="1.57"/>
     </joint>
     <joint name="${prefix}middle_joint2" type="revolute">
@@ -443,5 +443,5 @@
       <child link="${prefix}middle_link2"/>
       <axis xyz="0 1 0"/>
-      <limit lower="0" upper="1.6581" effort="1.2" velocity="1.57"/>
+      <limit lower="0" upper="1.666091" effort="1.2" velocity="1.57"/>
     </joint>
     <joint name="${prefix}middle_joint3" type="revolute">
@@ -450,5 +450,5 @@
       <child link="${prefix}middle_link3"/>
       <axis xyz="0 1 0"/>
-      <limit lower="0" upper="1.5533" effort="1.2" velocity="1.57"/>
+      <limit lower="0" upper="1.570796" effort="1.2" velocity="1.57"/>
     </joint>
     <joint name="${prefix}middle_joint4" type="revolute">
@@ -457,5 +457,5 @@
       <child link="${prefix}middle_link4"/>
       <axis xyz="0 1 0"/>
-      <limit lower="0" upper="1.6319" effort="1.2" velocity="1.57"/>
+      <limit lower="0" upper="1.739111" effort="1.2" velocity="1.57"/>  <!-- passive: q3 90° 에서 유도 (four-bar) -->
     </joint>
     <!-- ================================ ring finger ================================ -->
@@ -565,5 +565,5 @@
       <child link="${prefix}ring_link1"/>
       <axis xyz="0 1 0"/>
-      <limit lower="-0.5236" upper="0.5236" effort="1.2" velocity="1.57"/>
+      <limit lower="-0.479966" upper="0.479966" effort="1.2" velocity="1.57"/>
     </joint>
     <joint name="${prefix}ring_joint2" type="revolute">
@@ -572,5 +572,5 @@
       <child link="${prefix}ring_link2"/>
       <axis xyz="0 1 0"/>
-      <limit lower="0" upper="1.6581" effort="1.2" velocity="1.57"/>
+      <limit lower="0" upper="1.666091" effort="1.2" velocity="1.57"/>
     </joint>
     <joint name="${prefix}ring_joint3" type="revolute">
@@ -579,5 +579,5 @@
       <child link="${prefix}ring_link3"/>
       <axis xyz="0 1 0"/>
-      <limit lower="0" upper="1.5533" effort="1.2" velocity="1.57"/>
+      <limit lower="0" upper="1.570796" effort="1.2" velocity="1.57"/>
     </joint>
     <joint name="${prefix}ring_joint4" type="revolute">
@@ -586,5 +586,5 @@
       <child link="${prefix}ring_link4"/>
       <axis xyz="0 1 0"/>
-      <limit lower="0" upper="1.6319" effort="1.2" velocity="1.57"/>
+      <limit lower="0" upper="1.739111" effort="1.2" velocity="1.57"/>  <!-- passive: q3 90° 에서 유도 (four-bar) -->
     </joint>
     <!-- ================================ baby finger ================================ -->
@@ -694,5 +694,5 @@
       <child link="${prefix}baby_link1"/>
       <axis xyz="0 1 0"/>
-      <limit lower="-0.5236" upper="0.5236" effort="1.2" velocity="1.57"/>
+      <limit lower="-0.479966" upper="0.479966" effort="1.2" velocity="1.57"/>
     </joint>
     <joint name="${prefix}baby_joint2" type="revolute">
@@ -701,5 +701,5 @@
       <child link="${prefix}baby_link2"/>
       <axis xyz="0 1 0"/>
-      <limit lower="0" upper="1.6581" effort="1.2" velocity="1.57"/>
+      <limit lower="0" upper="1.666091" effort="1.2" velocity="1.57"/>
     </joint>
     <joint name="${prefix}baby_joint3" type="revolute">
@@ -708,5 +708,5 @@
       <child link="${prefix}baby_link3"/>
       <axis xyz="0 1 0"/>
-      <limit lower="0" upper="1.5533" effort="1.2" velocity="1.57"/>
+      <limit lower="0" upper="1.570796" effort="1.2" velocity="1.57"/>
     </joint>
     <joint name="${prefix}baby_joint4" type="revolute">
@@ -715,5 +715,5 @@
       <child link="${prefix}baby_link4"/>
       <axis xyz="0 1 0"/>
-      <limit lower="0" upper="1.6319" effort="1.2" velocity="1.57"/>
+      <limit lower="0" upper="1.739111" effort="1.2" velocity="1.57"/>  <!-- passive: q3 90° 에서 유도 (four-bar) -->
     </joint>
   </xacro:macro>
