Commit message: feat(description): Rebuild the hands from the 260918 CAD revision
The description held geometry from before the revision that added the
tactile pads, so the palm mass was 32 g short and the finger roots sat
8.9 mm too low. Nothing in the URDF said where a tactile pad was.

Both hands are regenerated from the SW2URDF export, with 17 tactile
links each on fixed joints. Meshes move to meshes/<side>_aidin_hand2/
and each file takes the name of the link it draws, so the left hand no
longer borrows the right hand's meshes through a negative scale. Joint
limits are the CAD values.

The RViz config drops a hardcoded link list that had gone stale, and
the control guide gains the slider method for sending joint commands.

File: aidin_hand2_description/urdf/aidin_hand2_left.urdf.xacro (robot description, xacro)
@@ -2,13 +2,7 @@
 <!--
   Hand-left macro for aidin_hand2.
-  GENERATED as the true geometric mirror of aidin_hand2_right.urdf.xacro across the
-  XZ plane (M = diag(1,-1,1), i.e. Y -> -Y).  Per-element rule:
-    - link/joint origin xyz : negate Y
-    - link/joint origin rpy : R' = M R M  (recomputed)
-    - inertia tensor        : ixy, iyz sign flipped (ixx/iyy/izz/ixz unchanged)
-    - joint axis            : a' = -M a
-    - mass / limit / effort / velocity : unchanged
-    - palm mesh             : body_right.STL -> body_left.STL
-    - finger mesh           : the shared STL, mirrored by a link-local Y scale
+  GENERATED from the SW2URDF export by dev/shared/scripts/build/sw2urdf-to-xacro.
+  Mesh files live under aidin_hand2_description/meshes/left_aidin_hand2/{visual,collision}/
+  and share the same filename across the two directories.
 -->
 <robot xmlns:xacro="http://www.ros.org/wiki/xacro">
@@ -24,50 +18,112 @@
     <link name="${prefix}hand_base_link">
       <inertial>
-        <origin xyz="0.00320138275084623 -0.000486961406823378 0.0551088066173012" rpy="0 0 0"/>
-        <mass value="0.224653931713756"/>
-        <inertia
-          ixx="0.0001829801686329" ixy="-5.97967829542247E-07" ixz="-2.90350893810316E-06"
-          iyy="9.92584141817906E-05" iyz="1.62408221940103E-06"
-          izz="0.000137495988458663"/>
-      </inertial>
-      <visual>
-        <origin xyz="0 0 0" rpy="0 0 0"/>
-        <geometry>
-          <mesh filename="package://aidin_hand2_description/meshes/visual/body_left.STL"/>
-        </geometry>
-        <material name="">
-          <color rgba="0.752941176470588 0.752941176470588 0.752941176470588 1"/>
-        </material>
-      </visual>
-      <collision>
-        <origin xyz="0 0 0" rpy="0 0 0"/>
-        <geometry>
-          <mesh filename="package://aidin_hand2_description/meshes/collision/body_left.STL"/>
-        </geometry>
-      </collision>
-    </link>
+        <origin xyz="-0.00112900319101962 -0.000654709257800466 0.0477993752418005" rpy="0 0 0"/>
+        <mass value="0.200555844551245"/>
+        <inertia
+          ixx="0.00018231692021459" ixy="-2.30409801745255E-07" ixz="-9.55605011249849E-07"
+          iyy="0.000110054551030555" iyz="4.54625088991344E-06"
+          izz="0.000150549981411924"/>
+      </inertial>
+      <visual>
+        <origin xyz="0 0 0" rpy="0 0 0"/>
+        <geometry>
+          <mesh filename="package://aidin_hand2_description/meshes/left_aidin_hand2/visual/left_hand_base_link.STL"/>
+        </geometry>
+        <material name="">
+          <color rgba="0.223529411764706 0.223529411764706 0.223529411764706 1"/>
+        </material>
+      </visual>
+      <collision>
+        <origin xyz="0 0 0" rpy="0 0 0"/>
+        <geometry>
+          <mesh filename="package://aidin_hand2_description/meshes/left_aidin_hand2/collision/left_hand_base_link.STL"/>
+        </geometry>
+      </collision>
+    </link>
+    <link name="${prefix}palm_tactile_top_link">
+      <inertial>
+        <origin xyz="0.000674762753468287 0.000606142354499798 0.0168891754218837" rpy="0 0 0"/>
+        <mass value="0.00740660791592135"/>
+        <inertia
+          ixx="5.31401179825433E-06" ixy="-3.38325185098855E-10" ixz="-2.1687309555648E-10"
+          iyy="7.98284716819682E-07" iyz="1.74718767974592E-09"
+          izz="4.51808635096857E-06"/>
+      </inertial>
+      <visual>
+        <origin xyz="0 0 0" rpy="0 0 0"/>
+        <geometry>
+          <mesh filename="package://aidin_hand2_description/meshes/left_aidin_hand2/visual/left_palm_tactile_top_link.STL"/>
+        </geometry>
+        <material name="">
+          <color rgba="0.274509803921569 0.274509803921569 0.274509803921569 1"/>
+        </material>
+      </visual>
+      <collision>
+        <origin xyz="0 0 0" rpy="0 0 0"/>
+        <geometry>
+          <mesh filename="package://aidin_hand2_description/meshes/left_aidin_hand2/collision/left_palm_tactile_top_link.STL"/>
+        </geometry>
+      </collision>
+    </link>
+    <link name="${prefix}palm_tactile_bottom_link">
+      <inertial>
+        <origin xyz="-0.0305 -0.0205 -0.0289" rpy="0 0 0"/>
+        <mass value="2.63186785647137E-09"/>
+        <inertia
+          ixx="7.49450015306718E-13" ixy="-1.57583383285962E-16" ixz="1.20748625558926E-16"
+          iyy="3.09128508139386E-13" iyz="-2.11408592851147E-14"
+          izz="4.44014404594315E-13"/>
+      </inertial>
+      <visual>
+        <origin xyz="0 0 0" rpy="0 0 0"/>
+        <geometry>
+          <mesh filename="package://aidin_hand2_description/meshes/left_aidin_hand2/visual/left_palm_tactile_bottom_link.STL"/>
+        </geometry>
+        <material name="">
+          <color rgba="0.274509803921569 0.274509803921569 0.274509803921569 1"/>
+        </material>
+      </visual>
+      <collision>
+        <origin xyz="0 0 0" rpy="0 0 0"/>
+        <geometry>
+          <mesh filename="package://aidin_hand2_description/meshes/left_aidin_hand2/collision/left_palm_tactile_bottom_link.STL"/>
+        </geometry>
+      </collision>
+    </link>
+    <joint name="${prefix}palm_tactile_top_joint" type="fixed">
+      <origin xyz="0.0305 0 0.0669" rpy="0 0 0"/>
+      <parent link="${prefix}hand_base_link"/>
+      <child link="${prefix}palm_tactile_top_link"/>
+      <axis xyz="0 0 0"/>
+    </joint>
+    <joint name="${prefix}palm_tactile_bottom_joint" type="fixed">
+      <origin xyz="0.0305 0.0205 0.0289" rpy="0 0 0"/>
+      <parent link="${prefix}hand_base_link"/>
+      <child link="${prefix}palm_tactile_bottom_link"/>
+      <axis xyz="0 0 0"/>
+    </joint>
     <!-- ============================== Thumb ============================= -->
     <link name="${prefix}thumb_link0">
       <inertial>
-        <origin xyz="-0.000530418447680113 -0.0181722170592327 -0.00309086613343537" rpy="0 0 0"/>
-        <mass value="0.0260533922416012"/>
-        <inertia
-          ixx="4.24619727662572E-06" ixy="3.63537752061735E-07" ixz="4.35690374733072E-08"
-          iyy="1.06435704456071E-06" iyz="-9.27840158955382E-07"
-          izz="4.06145127815098E-06"/>
-      </inertial>
-      <visual>
-        <origin xyz="0 0 0" rpy="0 0 0"/>
-        <geometry>
-          <mesh filename="package://aidin_hand2_description/meshes/visual/thumb_link0.STL" scale="1 -1 1"/>
-        </geometry>
-        <material name="">
-          <color rgba="1 1 1 1"/>
-        </material>
-      </visual>
-      <collision>
-        <origin xyz="0 0 0" rpy="0 0 0"/>
-        <geometry>
-          <mesh filename="package://aidin_hand2_description/meshes/collision/thumb_link0.STL" scale="1 -1 1"/>
+        <origin xyz="-2.04529594044107E-05 -0.0036917238386656 0.0215358561772485" rpy="0 0 0"/>
+        <mass value="0.0175117847223968"/>
+        <inertia
+          ixx="2.74153385446541E-06" ixy="-3.48140106171521E-09" ixz="1.15689831220349E-08"
+          iyy="2.61724678840433E-06" iyz="7.04056345733139E-07"
+          izz="6.42238676991707E-07"/>
+      </inertial>
+      <visual>
+        <origin xyz="0 0 0" rpy="0 0 0"/>
+        <geometry>
+          <mesh filename="package://aidin_hand2_description/meshes/left_aidin_hand2/visual/left_thumb_link0.STL"/>
+        </geometry>
+        <material name="">
+          <color rgba="0.223529411764706 0.223529411764706 0.223529411764706 1"/>
+        </material>
+      </visual>
+      <collision>
+        <origin xyz="0 0 0" rpy="0 0 0"/>
+        <geometry>
+          <mesh filename="package://aidin_hand2_description/meshes/left_aidin_hand2/collision/left_thumb_link0.STL"/>
         </geometry>
       </collision>
@@ -75,24 +131,24 @@
     <link name="${prefix}thumb_link1">
       <inertial>
-        <origin xyz="-2.89689407705074E-09 0 -6.93889390390723E-18" rpy="0 0 0"/>
-        <mass value="0.00168600740995136"/>
-        <inertia
-          ixx="1.51871371348108E-08" ixy="-1.39586728368323E-24" ixz="1.52834542866243E-24"
-          iyy="8.17450228480578E-09" iyz="-2.86124765907588E-14"
-          izz="1.20447607207831E-08"/>
-      </inertial>
-      <visual>
-        <origin xyz="0 0 0" rpy="0 0 0"/>
-        <geometry>
-          <mesh filename="package://aidin_hand2_description/meshes/visual/thumb_link1.STL" scale="1 -1 1"/>
-        </geometry>
-        <material name="">
-          <color rgba="0.752941176470588 0.752941176470588 0.752941176470588 1"/>
-        </material>
-      </visual>
-      <collision>
-        <origin xyz="0 0 0" rpy="0 0 0"/>
-        <geometry>
-          <mesh filename="package://aidin_hand2_description/meshes/collision/thumb_link1.STL" scale="1 -1 1"/>
+        <origin xyz="3.46944695195361E-18 0 -1.38777878078145E-17" rpy="0 0 0"/>
+        <mass value="0.00173685390848987"/>
+        <inertia
+          ixx="1.60398098537176E-08" ixy="3.87740912134232E-24" ixz="-7.85175347071819E-25"
+          iyy="8.83849653734709E-09" iyz="-6.72084247699335E-25"
+          izz="1.2667791817983E-08"/>
+      </inertial>
+      <visual>
+        <origin xyz="0 0 0" rpy="0 0 0"/>
+        <geometry>
+          <mesh filename="package://aidin_hand2_description/meshes/left_aidin_hand2/visual/left_thumb_link1.STL"/>
+        </geometry>
+        <material name="">
+          <color rgba="0.223529411764706 0.223529411764706 0.223529411764706 1"/>
+        </material>
+      </visual>
+      <collision>
+        <origin xyz="0 0 0" rpy="0 0 0"/>
+        <geometry>
+          <mesh filename="package://aidin_hand2_description/meshes/left_aidin_hand2/collision/left_thumb_link1.STL"/>
         </geometry>
       </collision>
@@ -100,24 +156,24 @@
     <link name="${prefix}thumb_link2">
       <inertial>
-        <origin xyz="0.000148107948271171 -0.00020287748317661 0.0400483513474308" rpy="0 0 0"/>
-        <mass value="0.0443650382155745"/>
-        <inertia
-          ixx="8.04809181854868E-06" ixy="-2.07341226978115E-08" ixz="4.86028773336942E-10"
-          iyy="6.58335865504048E-06" iyz="-1.15805857574675E-06"
-          izz="5.62089846720055E-06"/>
-      </inertial>
-      <visual>
-        <origin xyz="0 0 0" rpy="0 0 0"/>
-        <geometry>
-          <mesh filename="package://aidin_hand2_description/meshes/visual/thumb_link2.STL" scale="1 -1 1"/>
-        </geometry>
-        <material name="">
-          <color rgba="0.752941176470588 0.752941176470588 0.752941176470588 1"/>
-        </material>
-      </visual>
-      <collision>
-        <origin xyz="0 0 0" rpy="0 0 0"/>
-        <geometry>
-          <mesh filename="package://aidin_hand2_description/meshes/collision/thumb_link2.STL" scale="1 -1 1"/>
+        <origin xyz="2.72781485055433E-05 -0.0010633450190935 0.0366448131549096" rpy="0 0 0"/>
+        <mass value="0.0306656546978785"/>
+        <inertia
+          ixx="6.50266677995518E-06" ixy="8.67689746732147E-09" ixz="-1.88920869630403E-09"
+          iyy="7.52035679754067E-06" iyz="1.00843909703269E-07"
+          izz="4.07281004231722E-06"/>
+      </inertial>
+      <visual>
+        <origin xyz="0 0 0" rpy="0 0 0"/>
+        <geometry>
+          <mesh filename="package://aidin_hand2_description/meshes/left_aidin_hand2/visual/left_thumb_link2.STL"/>
+        </geometry>
+        <material name="">
+          <color rgba="0.223529411764706 0.223529411764706 0.223529411764706 1"/>
+        </material>
+      </visual>
+      <collision>
+        <origin xyz="0 0 0" rpy="0 0 0"/>
+        <geometry>
+          <mesh filename="package://aidin_hand2_description/meshes/left_aidin_hand2/collision/left_thumb_link2.STL"/>
         </geometry>
       </collision>
@@ -125,24 +181,24 @@
     <link name="${prefix}thumb_link3">
       <inertial>
-        <origin xyz="0.000587314896026189 -7.39809355690645E-05 0.0253022394365516" rpy="0 0 0"/>
-        <mass value="0.0187253772868473"/>
-        <inertia
-          ixx="2.4783907743346E-06" ixy="3.30382268553285E-08" ixz="1.60565367946041E-07"
-          iyy="2.80966458337564E-06" iyz="-5.85361301662048E-08"
-          izz="5.74868339605637E-07"/>
-      </inertial>
-      <visual>
-        <origin xyz="0 0 0" rpy="0 0 0"/>
-        <geometry>
-          <mesh filename="package://aidin_hand2_description/meshes/visual/thumb_link3.STL" scale="1 -1 1"/>
-        </geometry>
-        <material name="">
-          <color rgba="0.752941176470588 0.752941176470588 0.752941176470588 1"/>
-        </material>
-      </visual>
-      <collision>
-        <origin xyz="0 0 0" rpy="0 0 0"/>
-        <geometry>
-          <mesh filename="package://aidin_hand2_description/meshes/collision/thumb_link3.STL" scale="1 -1 1"/>
+        <origin xyz="6.3329481398873E-05 1.48616055370421E-06 0.0219809085256264" rpy="0 0 0"/>
+        <mass value="0.0201937490110632"/>
+        <inertia
+          ixx="2.04793315056244E-06" ixy="-4.26002969599587E-08" ixz="-2.95529913508848E-07"
+          iyy="2.43224674957065E-06" iyz="-1.14296385060062E-08"
+          izz="6.38342422611227E-07"/>
+      </inertial>
+      <visual>
+        <origin xyz="0 0 0" rpy="0 0 0"/>
+        <geometry>
+          <mesh filename="package://aidin_hand2_description/meshes/left_aidin_hand2/visual/left_thumb_link3.STL"/>
+        </geometry>
+        <material name="">
+          <color rgba="0.223529411764706 0.223529411764706 0.223529411764706 1"/>
+        </material>
+      </visual>
+      <collision>
+        <origin xyz="0 0 0" rpy="0 0 0"/>
+        <geometry>
+          <mesh filename="package://aidin_hand2_description/meshes/left_aidin_hand2/collision/left_thumb_link3.STL"/>
         </geometry>
       </collision>
@@ -150,40 +206,115 @@
     <link name="${prefix}thumb_link4">
       <inertial>
-        <origin xyz="0.000633912547249024 7.69891472292977E-06 0.0132530698716445" rpy="0 0 0"/>
-        <mass value="0.0140770241572427"/>
-        <inertia
-          ixx="9.93116317288254E-07" ixy="3.21252609854791E-08" ixz="4.62754443985299E-08"
-          iyy="7.85919048408442E-07" iyz="-1.10106687992887E-07"
-          izz="5.1923881092419E-07"/>
-      </inertial>
-      <visual>
-        <origin xyz="0 0 0" rpy="0 0 0"/>
-        <geometry>
-          <mesh filename="package://aidin_hand2_description/meshes/visual/thumb_link4.STL" scale="1 -1 1"/>
-        </geometry>
-        <material name="">
-          <color rgba="0.752941176470588 0.752941176470588 0.752941176470588 1"/>
-        </material>
-      </visual>
-      <collision>
-        <origin xyz="0 0 0" rpy="0 0 0"/>
-        <geometry>
-          <mesh filename="package://aidin_hand2_description/meshes/collision/thumb_link4.STL" scale="1 -1 1"/>
+        <origin xyz="-8.13507476343303E-05 6.53313213021603E-06 0.0125489245833013" rpy="0 0 0"/>
+        <mass value="0.0111473616667527"/>
+        <inertia
+          ixx="8.82920873346288E-07" ixy="-3.57279017168599E-08" ixz="7.22553841879569E-08"
+          iyy="7.73222675658295E-07" iyz="1.24168999943475E-07"
+          izz="4.20743520963829E-07"/>
+      </inertial>
+      <visual>
+        <origin xyz="0 0 0" rpy="0 0 0"/>
+        <geometry>
+          <mesh filename="package://aidin_hand2_description/meshes/left_aidin_hand2/visual/left_thumb_link4.STL"/>
+        </geometry>
+        <material name="">
+          <color rgba="0.223529411764706 0.223529411764706 0.223529411764706 1"/>
+        </material>
+      </visual>
+      <collision>
+        <origin xyz="0 0 0" rpy="0 0 0"/>
+        <geometry>
+          <mesh filename="package://aidin_hand2_description/meshes/left_aidin_hand2/collision/left_thumb_link4.STL"/>
+        </geometry>
+      </collision>
+    </link>
+    <link name="${prefix}thumb_tactile_link2">
+      <inertial>
+        <origin xyz="0.00324776330394302 0.000160674203724266 0.0105206453579296" rpy="0 0 0"/>
+        <mass value="0.00197158860531171"/>
+        <inertia
+          ixx="1.1095086185982E-07" ixy="7.73965616235978E-10" ixz="9.55396920752724E-11"
+          iyy="7.72325483152603E-08" iyz="6.88587177292641E-11"
+          izz="4.67035800534061E-08"/>
+      </inertial>
+      <visual>
+        <origin xyz="0 0 0" rpy="0 0 0"/>
+        <geometry>
+          <mesh filename="package://aidin_hand2_description/meshes/left_aidin_hand2/visual/left_thumb_tactile_link2.STL"/>
+        </geometry>
+        <material name="">
+          <color rgba="0.274509803921569 0.274509803921569 0.274509803921569 1"/>
+        </material>
+      </visual>
+      <collision>
+        <origin xyz="0 0 0" rpy="0 0 0"/>
+        <geometry>
+          <mesh filename="package://aidin_hand2_description/meshes/left_aidin_hand2/collision/left_thumb_tactile_link2.STL"/>
+        </geometry>
+      </collision>
+    </link>
+    <link name="${prefix}thumb_tactile_link3">
+      <inertial>
+        <origin xyz="0.00402433958626983 3.63916216605809E-10 0.00549999923047306" rpy="0 0 0"/>
+        <mass value="6.39299774482251E-10"/>
+        <inertia
+          ixx="3.73656390346653E-14" ixy="-1.44586493401505E-21" ixz="-1.64162584188864E-20"
+          iyy="1.02586581914774E-14" iyz="1.38967187941937E-19"
+          izz="3.14387262901213E-14"/>
+      </inertial>
+      <visual>
+        <origin xyz="0 0 0" rpy="0 0 0"/>
+        <geometry>
+          <mesh filename="package://aidin_hand2_description/meshes/left_aidin_hand2/visual/left_thumb_tactile_link3.STL"/>
+        </geometry>
+        <material name="">
+          <color rgba="0.274509803921569 0.274509803921569 0.274509803921569 1"/>
+        </material>
+      </visual>
+      <collision>
+        <origin xyz="0 0 0" rpy="0 0 0"/>
+        <geometry>
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