Commit message: feat(description): Rebuild the hands from the 260918 CAD revision
The description held geometry from before the revision that added the
tactile pads, so the palm mass was 32 g short and the finger roots sat
8.9 mm too low. Nothing in the URDF said where a tactile pad was.

Both hands are regenerated from the SW2URDF export, with 17 tactile
links each on fixed joints. Meshes move to meshes/<side>_aidin_hand2/
and each file takes the name of the link it draws, so the left hand no
longer borrows the right hand's meshes through a negative scale. Joint
limits are the CAD values.

The RViz config drops a hardcoded link list that had gone stale, and
the control guide gains the slider method for sending joint commands.

File: aidin_hand2_description/urdf/aidin_hand2_right.urdf.xacro (robot description, xacro)
@@ -2,6 +2,7 @@
 <!--
   Hand-right macro for aidin_hand2.
-  Mesh files live under aidin_hand2_description/meshes/{visual,collision}/
-  and share the same filename across visual/ and collision/ directories.
+  GENERATED from the SW2URDF export by dev/shared/scripts/build/sw2urdf-to-xacro.
+  Mesh files live under aidin_hand2_description/meshes/right_aidin_hand2/{visual,collision}/
+  and share the same filename across the two directories.
 -->
 <robot xmlns:xacro="http://www.ros.org/wiki/xacro">
@@ -17,50 +18,112 @@
     <link name="${prefix}hand_base_link">
       <inertial>
-        <origin xyz="0.00320138275084623 0.000486961406823378 0.0551088066173012" rpy="0 0 0"/>
-        <mass value="0.224653931713756"/>
-        <inertia
-          ixx="0.0001829801686329" ixy="5.97967829542247E-07" ixz="-2.90350893810316E-06"
-          iyy="9.92584141817906E-05" iyz="-1.62408221940103E-06"
-          izz="0.000137495988458663"/>
-      </inertial>
-      <visual>
-        <origin xyz="0 0 0" rpy="0 0 0"/>
-        <geometry>
-          <mesh filename="package://aidin_hand2_description/meshes/visual/body_right.STL"/>
-        </geometry>
-        <material name="">
-          <color rgba="0.752941176470588 0.752941176470588 0.752941176470588 1"/>
-        </material>
-      </visual>
-      <collision>
-        <origin xyz="0 0 0" rpy="0 0 0"/>
-        <geometry>
-          <mesh filename="package://aidin_hand2_description/meshes/collision/body_right.STL"/>
-        </geometry>
-      </collision>
-    </link>
+        <origin xyz="-6.24179943675983E-05 0.000367827113016154 0.0458864934845128" rpy="0 0 0"/>
+        <mass value="0.256337522909554"/>
+        <inertia
+          ixx="0.000237812316010346" ixy="9.54719046016524E-07" ixz="-1.13448821855029E-06"
+          iyy="0.00012638529968063" iyz="-5.78438894115108E-06"
+          izz="0.000195591173374432"/>
+      </inertial>
+      <visual>
+        <origin xyz="0 0 0" rpy="0 0 0"/>
+        <geometry>
+          <mesh filename="package://aidin_hand2_description/meshes/right_aidin_hand2/visual/right_hand_base_link.STL"/>
+        </geometry>
+        <material name="">
+          <color rgba="0.223529411764706 0.223529411764706 0.223529411764706 1"/>
+        </material>
+      </visual>
+      <collision>
+        <origin xyz="0 0 0" rpy="0 0 0"/>
+        <geometry>
+          <mesh filename="package://aidin_hand2_description/meshes/right_aidin_hand2/collision/right_hand_base_link.STL"/>
+        </geometry>
+      </collision>
+    </link>
+    <link name="${prefix}palm_tactile_top_link">
+      <inertial>
+        <origin xyz="0.000674762753468287 0.000606142354499799 0.0168891754218837" rpy="0 0 0"/>
+        <mass value="0.00740660791592135"/>
+        <inertia
+          ixx="5.31401179825433E-06" ixy="-3.38325185098854E-10" ixz="-2.1687309555648E-10"
+          iyy="7.98284716819682E-07" iyz="1.74718767974592E-09"
+          izz="4.51808635096857E-06"/>
+      </inertial>
+      <visual>
+        <origin xyz="0 0 0" rpy="0 0 0"/>
+        <geometry>
+          <mesh filename="package://aidin_hand2_description/meshes/right_aidin_hand2/visual/right_palm_tactile_top_link.STL"/>
+        </geometry>
+        <material name="">
+          <color rgba="0.274509803921569 0.274509803921569 0.274509803921569 1"/>
+        </material>
+      </visual>
+      <collision>
+        <origin xyz="0 0 0" rpy="0 0 0"/>
+        <geometry>
+          <mesh filename="package://aidin_hand2_description/meshes/right_aidin_hand2/collision/right_palm_tactile_top_link.STL"/>
+        </geometry>
+      </collision>
+    </link>
+    <link name="${prefix}palm_tactile_bottom_link">
+      <inertial>
+        <origin xyz="0.000649300878208026 0.000641439582478615 0.0169329552007083" rpy="0 0 0"/>
+        <mass value="0.00310671585401556"/>
+        <inertia
+          ixx="9.07160891349656E-07" ixy="-4.55727810648528E-11" ixz="-3.96752423296767E-11"
+          iyy="3.73671638314401E-07" iyz="2.86219742499054E-08"
+          izz="5.34403556862556E-07"/>
+      </inertial>
+      <visual>
+        <origin xyz="0 0 0" rpy="0 0 0"/>
+        <geometry>
+          <mesh filename="package://aidin_hand2_description/meshes/right_aidin_hand2/visual/right_palm_tactile_bottom_link.STL"/>
+        </geometry>
+        <material name="">
+          <color rgba="0.274509803921569 0.274509803921569 0.274509803921569 1"/>
+        </material>
+      </visual>
+      <collision>
+        <origin xyz="0 0 0" rpy="0 0 0"/>
+        <geometry>
+          <mesh filename="package://aidin_hand2_description/meshes/right_aidin_hand2/collision/right_palm_tactile_bottom_link.STL"/>
+        </geometry>
+      </collision>
+    </link>
+    <joint name="${prefix}palm_tactile_top_joint" type="fixed">
+      <origin xyz="0.0305 0 0.0669" rpy="0 0 0"/>
+      <parent link="${prefix}hand_base_link"/>
+      <child link="${prefix}palm_tactile_top_link"/>
+      <axis xyz="0 0 0"/>
+    </joint>
+    <joint name="${prefix}palm_tactile_bottom_joint" type="fixed">
+      <origin xyz="0.0305 -0.0205 0.0289" rpy="0 0 0"/>
+      <parent link="${prefix}hand_base_link"/>
+      <child link="${prefix}palm_tactile_bottom_link"/>
+      <axis xyz="0 0 0"/>
+    </joint>
     <!-- ============================== Thumb ============================= -->
     <link name="${prefix}thumb_link0">
       <inertial>
-        <origin xyz="-0.000530418447680113 0.0181722170592327 -0.00309086613343537" rpy="0 0 0"/>
-        <mass value="0.0260533922416012"/>
-        <inertia
-          ixx="4.24619727662572E-06" ixy="-3.63537752061735E-07" ixz="4.35690374733072E-08"
-          iyy="1.06435704456071E-06" iyz="9.27840158955382E-07"
-          izz="4.06145127815098E-06"/>
-      </inertial>
-      <visual>
-        <origin xyz="0 0 0" rpy="0 0 0"/>
-        <geometry>
-          <mesh filename="package://aidin_hand2_description/meshes/visual/thumb_link0.STL"/>
-        </geometry>
-        <material name="">
-          <color rgba="1 1 1 1"/>
-        </material>
-      </visual>
-      <collision>
-        <origin xyz="0 0 0" rpy="0 0 0"/>
-        <geometry>
-          <mesh filename="package://aidin_hand2_description/meshes/collision/thumb_link0.STL"/>
+        <origin xyz="2.04529950085935E-05 0.00369172383122075 0.0215358560719203" rpy="0 0 0"/>
+        <mass value="0.0175117847643855"/>
+        <inertia
+          ixx="2.74153386147205E-06" ixy="-3.48140054036223E-09" ixz="-1.15689797191921E-08"
+          iyy="2.61724679529738E-06" iyz="-7.04056347941746E-07"
+          izz="6.422386783828E-07"/>
+      </inertial>
+      <visual>
+        <origin xyz="0 0 0" rpy="0 0 0"/>
+        <geometry>
+          <mesh filename="package://aidin_hand2_description/meshes/right_aidin_hand2/visual/right_thumb_link0.STL"/>
+        </geometry>
+        <material name="">
+          <color rgba="0.223529411764706 0.223529411764706 0.223529411764706 1"/>
+        </material>
+      </visual>
+      <collision>
+        <origin xyz="0 0 0" rpy="0 0 0"/>
+        <geometry>
+          <mesh filename="package://aidin_hand2_description/meshes/right_aidin_hand2/collision/right_thumb_link0.STL"/>
         </geometry>
       </collision>
@@ -68,24 +131,24 @@
     <link name="${prefix}thumb_link1">
       <inertial>
-        <origin xyz="-2.89689407705074E-09 0 -6.93889390390723E-18" rpy="0 0 0"/>
-        <mass value="0.00168600740995136"/>
-        <inertia
-          ixx="1.51871371348108E-08" ixy="1.39586728368323E-24" ixz="1.52834542866243E-24"
-          iyy="8.17450228480578E-09" iyz="2.86124765907588E-14"
-          izz="1.20447607207831E-08"/>
-      </inertial>
-      <visual>
-        <origin xyz="0 0 0" rpy="0 0 0"/>
-        <geometry>
-          <mesh filename="package://aidin_hand2_description/meshes/visual/thumb_link1.STL"/>
-        </geometry>
-        <material name="">
-          <color rgba="0.752941176470588 0.752941176470588 0.752941176470588 1"/>
-        </material>
-      </visual>
-      <collision>
-        <origin xyz="0 0 0" rpy="0 0 0"/>
-        <geometry>
-          <mesh filename="package://aidin_hand2_description/meshes/collision/thumb_link1.STL"/>
+        <origin xyz="6.93889390390723E-18 0 1.38777878078145E-17" rpy="0 0 0"/>
+        <mass value="0.00173685390848986"/>
+        <inertia
+          ixx="1.60398098537176E-08" ixy="3.10192729707385E-24" ixz="1.053362811298E-24"
+          iyy="8.83849653734704E-09" iyz="-1.03397576569128E-25"
+          izz="1.26677918179829E-08"/>
+      </inertial>
+      <visual>
+        <origin xyz="0 0 0" rpy="0 0 0"/>
+        <geometry>
+          <mesh filename="package://aidin_hand2_description/meshes/right_aidin_hand2/visual/right_thumb_link1.STL"/>
+        </geometry>
+        <material name="">
+          <color rgba="0.223529411764706 0.223529411764706 0.223529411764706 1"/>
+        </material>
+      </visual>
+      <collision>
+        <origin xyz="0 0 0" rpy="0 0 0"/>
+        <geometry>
+          <mesh filename="package://aidin_hand2_description/meshes/right_aidin_hand2/collision/right_thumb_link1.STL"/>
         </geometry>
       </collision>
@@ -93,24 +156,24 @@
     <link name="${prefix}thumb_link2">
       <inertial>
-        <origin xyz="0.000148107948271171 0.00020287748317661 0.0400483513474308" rpy="0 0 0"/>
-        <mass value="0.0443650382155745"/>
-        <inertia
-          ixx="8.04809181854868E-06" ixy="2.07341226978115E-08" ixz="4.86028773336942E-10"
-          iyy="6.58335865504048E-06" iyz="1.15805857574675E-06"
-          izz="5.62089846720055E-06"/>
-      </inertial>
-      <visual>
-        <origin xyz="0 0 0" rpy="0 0 0"/>
-        <geometry>
-          <mesh filename="package://aidin_hand2_description/meshes/visual/thumb_link2.STL"/>
-        </geometry>
-        <material name="">
-          <color rgba="0.752941176470588 0.752941176470588 0.752941176470588 1"/>
-        </material>
-      </visual>
-      <collision>
-        <origin xyz="0 0 0" rpy="0 0 0"/>
-        <geometry>
-          <mesh filename="package://aidin_hand2_description/meshes/collision/thumb_link2.STL"/>
+        <origin xyz="-2.72615030864343E-05 0.00106339106438241 0.0366448387885369" rpy="0 0 0"/>
+        <mass value="0.0306657105866884"/>
+        <inertia
+          ixx="6.50268004872161E-06" ixy="8.66958831618096E-09" ixz="1.87736911357994E-09"
+          iyy="7.52036467930933E-06" iyz="-1.00852489658317E-07"
+          izz="4.07281966959805E-06"/>
+      </inertial>
+      <visual>
+        <origin xyz="0 0 0" rpy="0 0 0"/>
+        <geometry>
+          <mesh filename="package://aidin_hand2_description/meshes/right_aidin_hand2/visual/right_thumb_link2.STL"/>
+        </geometry>
+        <material name="">
+          <color rgba="0.223529411764706 0.223529411764706 0.223529411764706 1"/>
+        </material>
+      </visual>
+      <collision>
+        <origin xyz="0 0 0" rpy="0 0 0"/>
+        <geometry>
+          <mesh filename="package://aidin_hand2_description/meshes/right_aidin_hand2/collision/right_thumb_link2.STL"/>
         </geometry>
       </collision>
@@ -118,24 +181,24 @@
     <link name="${prefix}thumb_link3">
       <inertial>
-        <origin xyz="0.000587314896026189 7.39809355690645E-05 0.0253022394365516" rpy="0 0 0"/>
-        <mass value="0.0187253772868473"/>
-        <inertia
-          ixx="2.4783907743346E-06" ixy="-3.30382268553285E-08" ixz="1.60565367946041E-07"
-          iyy="2.80966458337564E-06" iyz="5.85361301662048E-08"
-          izz="5.74868339605637E-07"/>
-      </inertial>
-      <visual>
-        <origin xyz="0 0 0" rpy="0 0 0"/>
-        <geometry>
-          <mesh filename="package://aidin_hand2_description/meshes/visual/thumb_link3.STL"/>
-        </geometry>
-        <material name="">
-          <color rgba="0.752941176470588 0.752941176470588 0.752941176470588 1"/>
-        </material>
-      </visual>
-      <collision>
-        <origin xyz="0 0 0" rpy="0 0 0"/>
-        <geometry>
-          <mesh filename="package://aidin_hand2_description/meshes/collision/thumb_link3.STL"/>
+        <origin xyz="6.33301090034559E-05 1.48829310408008E-06 0.0219809071453854" rpy="0 0 0"/>
+        <mass value="0.0201937467097963"/>
+        <inertia
+          ixx="2.0479328420402E-06" ixy="-4.26003484126146E-08" ixz="-2.95530046143824E-07"
+          iyy="2.43224635749665E-06" iyz="-1.14295380455757E-08"
+          izz="6.38342358784111E-07"/>
+      </inertial>
+      <visual>
+        <origin xyz="0 0 0" rpy="0 0 0"/>
+        <geometry>
+          <mesh filename="package://aidin_hand2_description/meshes/right_aidin_hand2/visual/right_thumb_link3.STL"/>
+        </geometry>
+        <material name="">
+          <color rgba="0.223529411764706 0.223529411764706 0.223529411764706 1"/>
+        </material>
+      </visual>
+      <collision>
+        <origin xyz="0 0 0" rpy="0 0 0"/>
+        <geometry>
+          <mesh filename="package://aidin_hand2_description/meshes/right_aidin_hand2/collision/right_thumb_link3.STL"/>
         </geometry>
       </collision>
@@ -143,40 +206,115 @@
     <link name="${prefix}thumb_link4">
       <inertial>
-        <origin xyz="0.000633912547249024 -7.69891472292977E-06 0.0132530698716445" rpy="0 0 0"/>
-        <mass value="0.0140770241572427"/>
-        <inertia
-          ixx="9.93116317288254E-07" ixy="-3.21252609854791E-08" ixz="4.62754443985299E-08"
-          iyy="7.85919048408442E-07" iyz="1.10106687992887E-07"
-          izz="5.1923881092419E-07"/>
-      </inertial>
-      <visual>
-        <origin xyz="0 0 0" rpy="0 0 0"/>
-        <geometry>
-          <mesh filename="package://aidin_hand2_description/meshes/visual/thumb_link4.STL"/>
-        </geometry>
-        <material name="">
-          <color rgba="0.752941176470588 0.752941176470588 0.752941176470588 1"/>
-        </material>
-      </visual>
-      <collision>
-        <origin xyz="0 0 0" rpy="0 0 0"/>
-        <geometry>
-          <mesh filename="package://aidin_hand2_description/meshes/collision/thumb_link4.STL"/>
+        <origin xyz="-8.13446157346756E-05 6.52203873742138E-06 0.0125488821785456" rpy="0 0 0"/>
+        <mass value="0.0111473427993758"/>
+        <inertia
+          ixx="8.82913361575911E-07" ixy="-3.57279330642873E-08" ixz="7.22548346536885E-08"
+          iyy="7.73215672454338E-07" iyz="1.24169841486205E-07"
+          izz="4.20743285569156E-07"/>
+      </inertial>
+      <visual>
+        <origin xyz="0 0 0" rpy="0 0 0"/>
+        <geometry>
+          <mesh filename="package://aidin_hand2_description/meshes/right_aidin_hand2/visual/right_thumb_link4.STL"/>
+        </geometry>
+        <material name="">
+          <color rgba="0.223529411764706 0.223529411764706 0.223529411764706 1"/>
+        </material>
+      </visual>
+      <collision>
+        <origin xyz="0 0 0" rpy="0 0 0"/>
+        <geometry>
+          <mesh filename="package://aidin_hand2_description/meshes/right_aidin_hand2/collision/right_thumb_link4.STL"/>
+        </geometry>
+      </collision>
+    </link>
+    <link name="${prefix}thumb_tactile_link2">
+      <inertial>
+        <origin xyz="0.00324776330394289 0.000160674216404193 0.0105206453633945" rpy="0 0 0"/>
+        <mass value="0.00197158860531087"/>
+        <inertia
+          ixx="1.10950861851881E-07" ixy="7.73967282273235E-10" ixz="9.55393797994464E-11"
+          iyy="7.72325483159031E-08" iyz="6.88587168681137E-11"
+          izz="4.67035800448894E-08"/>
+      </inertial>
+      <visual>
+        <origin xyz="0 0 0" rpy="0 0 0"/>
+        <geometry>
+          <mesh filename="package://aidin_hand2_description/meshes/right_aidin_hand2/visual/right_thumb_tactile_link2.STL"/>
+        </geometry>
+        <material name="">
+          <color rgba="0.274509803921569 0.274509803921569 0.274509803921569 1"/>
+        </material>
+      </visual>
+      <collision>
+        <origin xyz="0 0 0" rpy="0 0 0"/>
+        <geometry>
+          <mesh filename="package://aidin_hand2_description/meshes/right_aidin_hand2/collision/right_thumb_tactile_link2.STL"/>
+        </geometry>
+      </collision>
+    </link>
+    <link name="${prefix}thumb_tactile_link3">
+      <inertial>
+        <origin xyz="0.00402433958627001 3.66332533752178E-10 0.00549999922564851" rpy="0 0 0"/>
+        <mass value="6.3929977448218E-10"/>
+        <inertia
+          ixx="3.73656390341158E-14" ixy="-1.22419212705524E-21" ixz="-1.64403808786588E-20"
+          iyy="1.02586581912415E-14" iyz="1.38966805138209E-19"
+          izz="3.14387262898125E-14"/>
+      </inertial>
+      <visual>
+        <origin xyz="0 0 0" rpy="0 0 0"/>
+        <geometry>
+          <mesh filename="package://aidin_hand2_description/meshes/right_aidin_hand2/visual/right_thumb_tactile_link3.STL"/>
+        </geometry>
+        <material name="">
+          <color rgba="0.274509803921569 0.274509803921569 0.274509803921569 1"/>
+        </material>
+      </visual>
+      <collision>
+        <origin xyz="0 0 0" rpy="0 0 0"/>
+        <geometry>
+          <mesh filename="package://aidin_hand2_description/meshes/right_aidin_hand2/collision/right_thumb_tactile_link3.STL"/>
+        </geometry>
+      </collision>
+    </link>
+    <link name="${prefix}thumb_tactile_link4">
+      <inertial>
+        <origin xyz="0.00570492025683314 1.650514917656E-07 0.00947907082860006" rpy="0 0 0"/>
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