Commit message: refactor(description): Number palm tactile frames
The description was the only place calling the two palm boards top
and bottom. Every reading that comes off them is numbered: the
tactile_palm1_upper, tactile_palm1_lower and tactile_palm2 arrays in
HandState, and the palm1_upper_, palm1_lower_ and palm2_ interfaces
on the palm_sensor component. Nothing tied the frame a contact was
drawn in to the array it came from.

The new names also follow the {side}_{finger}_tactile_link{2,3,4}
the fingers already use.

File: aidin_hand2_description/urdf/aidin_hand2_left.urdf (robot description, URDF)
Before this commit: robot aidin_hand2_left, 39 links, 38 joints
Links:
- removed link left_palm_tactile_bottom_link
- removed link left_palm_tactile_top_link
- added link left_palm1_tactile_link, mass 0.00740660791592135; collision mesh filename=../meshes/left_aidin_hand2/collision/left_palm1_tactile_lin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; visual mesh filename=../meshes/left_aidin_hand2/visual/left_palm1_tactile_link.S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
- added link left_palm2_tactile_link, mass 2.63186785647137E-09; collision mesh filename=../meshes/left_aidin_hand2/collision/left_palm2_tactile_lin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; visual mesh filename=../meshes/left_aidin_hand2/visual/left_palm2_tactile_link.S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
Joints:
- removed joint left_palm_tactile_bottom_joint
- removed joint left_palm_tactile_top_joint
- added joint left_palm1_tactile_joint: type fixed, parent left_hand_base_link, child left_palm1_tactile_link, origin xyz=0.0305 0 0.0669 rpy=0 0 0, axis 0 0 0
- added joint left_palm2_tactile_joint: type fixed, parent left_hand_base_link, child left_palm2_tactile_link, origin xyz=0.0305 0.0205 0.0289 rpy=0 0 0, axis 0 0 0

File: aidin_hand2_description/urdf/aidin_hand2_right.urdf (robot description, URDF)
Before this commit: robot aidin_hand2_right, 39 links, 38 joints
Links:
- removed link right_palm_tactile_bottom_link
- removed link right_palm_tactile_top_link
- added link right_palm1_tactile_link, mass 0.00740660791592135; collision mesh filename=../meshes/right_aidin_hand2/collision/right_palm1_tactile_l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; visual mesh filename=../meshes/right_aidin_hand2/visual/right_palm1_tactile_link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
- added link right_palm2_tactile_link, mass 0.00310671585401556; collision mesh filename=../meshes/right_aidin_hand2/collision/right_palm2_tactile_l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; visual mesh filename=../meshes/right_aidin_hand2/visual/right_palm2_tactile_link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
Joints:
- removed joint right_palm_tactile_bottom_joint
- removed joint right_palm_tactile_top_joint
- added joint right_palm1_tactile_joint: type fixed, parent right_hand_base_link, child right_palm1_tactile_link, origin xyz=0.0305 0 0.0669 rpy=0 0 0, axis 0 0 0
- added joint right_palm2_tactile_joint: type fixed, parent right_hand_base_link, child right_palm2_tactile_link, origin xyz=0.0305 -0.0205 0.0289 rpy=0 0 0, axis 0 0 0

File: aidin_hand2_description/xacro/aidin_hand2_left.urdf.xacro (robot description, xacro)
@@ -41,5 +41,5 @@
       </collision>
     </link>
-    <link name="${prefix}palm_tactile_top_link">
+    <link name="${prefix}palm1_tactile_link">
       <inertial>
         <origin xyz="0.000674762753468287 0.000606142354499798 0.0168891754218837" rpy="0 0 0"/>
@@ -53,18 +53,18 @@
         <origin xyz="0 0 0" rpy="0 0 0"/>
         <geometry>
-          <mesh filename="package://aidin_hand2_description/meshes/left_aidin_hand2/visual/left_palm_tactile_top_link.STL"/>
-        </geometry>
-        <material name="">
-          <color rgba="0.274509803921569 0.274509803921569 0.274509803921569 1"/>
-        </material>
-      </visual>
-      <collision>
-        <origin xyz="0 0 0" rpy="0 0 0"/>
-        <geometry>
-          <mesh filename="package://aidin_hand2_description/meshes/left_aidin_hand2/collision/left_palm_tactile_top_link.STL"/>
-        </geometry>
-      </collision>
-    </link>
-    <link name="${prefix}palm_tactile_bottom_link">
+          <mesh filename="package://aidin_hand2_description/meshes/left_aidin_hand2/visual/left_palm1_tactile_link.STL"/>
+        </geometry>
+        <material name="">
+          <color rgba="0.274509803921569 0.274509803921569 0.274509803921569 1"/>
+        </material>
+      </visual>
+      <collision>
+        <origin xyz="0 0 0" rpy="0 0 0"/>
+        <geometry>
+          <mesh filename="package://aidin_hand2_description/meshes/left_aidin_hand2/collision/left_palm1_tactile_link.STL"/>
+        </geometry>
+      </collision>
+    </link>
+    <link name="${prefix}palm2_tactile_link">
       <inertial>
         <origin xyz="-0.0305 -0.0205 -0.0289" rpy="0 0 0"/>
@@ -78,27 +78,27 @@
         <origin xyz="0 0 0" rpy="0 0 0"/>
         <geometry>
-          <mesh filename="package://aidin_hand2_description/meshes/left_aidin_hand2/visual/left_palm_tactile_bottom_link.STL"/>
-        </geometry>
-        <material name="">
-          <color rgba="0.274509803921569 0.274509803921569 0.274509803921569 1"/>
-        </material>
-      </visual>
-      <collision>
-        <origin xyz="0 0 0" rpy="0 0 0"/>
-        <geometry>
-          <mesh filename="package://aidin_hand2_description/meshes/left_aidin_hand2/collision/left_palm_tactile_bottom_link.STL"/>
-        </geometry>
-      </collision>
-    </link>
-    <joint name="${prefix}palm_tactile_top_joint" type="fixed">
+          <mesh filename="package://aidin_hand2_description/meshes/left_aidin_hand2/visual/left_palm2_tactile_link.STL"/>
+        </geometry>
+        <material name="">
+          <color rgba="0.274509803921569 0.274509803921569 0.274509803921569 1"/>
+        </material>
+      </visual>
+      <collision>
+        <origin xyz="0 0 0" rpy="0 0 0"/>
+        <geometry>
+          <mesh filename="package://aidin_hand2_description/meshes/left_aidin_hand2/collision/left_palm2_tactile_link.STL"/>
+        </geometry>
+      </collision>
+    </link>
+    <joint name="${prefix}palm1_tactile_joint" type="fixed">
       <origin xyz="0.0305 0 0.0669" rpy="0 0 0"/>
       <parent link="${prefix}hand_base_link"/>
-      <child link="${prefix}palm_tactile_top_link"/>
-      <axis xyz="0 0 0"/>
-    </joint>
-    <joint name="${prefix}palm_tactile_bottom_joint" type="fixed">
+      <child link="${prefix}palm1_tactile_link"/>
+      <axis xyz="0 0 0"/>
+    </joint>
+    <joint name="${prefix}palm2_tactile_joint" type="fixed">
       <origin xyz="0.0305 0.0205 0.0289" rpy="0 0 0"/>
       <parent link="${prefix}hand_base_link"/>
-      <child link="${prefix}palm_tactile_bottom_link"/>
+      <child link="${prefix}palm2_tactile_link"/>
       <axis xyz="0 0 0"/>
     </joint>

File: aidin_hand2_description/xacro/aidin_hand2_right.urdf.xacro (robot description, xacro)
@@ -41,5 +41,5 @@
       </collision>
     </link>
-    <link name="${prefix}palm_tactile_top_link">
+    <link name="${prefix}palm1_tactile_link">
       <inertial>
         <origin xyz="0.000674762753468287 0.000606142354499799 0.0168891754218837" rpy="0 0 0"/>
@@ -53,18 +53,18 @@
         <origin xyz="0 0 0" rpy="0 0 0"/>
         <geometry>
-          <mesh filename="package://aidin_hand2_description/meshes/right_aidin_hand2/visual/right_palm_tactile_top_link.STL"/>
-        </geometry>
-        <material name="">
-          <color rgba="0.274509803921569 0.274509803921569 0.274509803921569 1"/>
-        </material>
-      </visual>
-      <collision>
-        <origin xyz="0 0 0" rpy="0 0 0"/>
-        <geometry>
-          <mesh filename="package://aidin_hand2_description/meshes/right_aidin_hand2/collision/right_palm_tactile_top_link.STL"/>
-        </geometry>
-      </collision>
-    </link>
-    <link name="${prefix}palm_tactile_bottom_link">
+          <mesh filename="package://aidin_hand2_description/meshes/right_aidin_hand2/visual/right_palm1_tactile_link.STL"/>
+        </geometry>
+        <material name="">
+          <color rgba="0.274509803921569 0.274509803921569 0.274509803921569 1"/>
+        </material>
+      </visual>
+      <collision>
+        <origin xyz="0 0 0" rpy="0 0 0"/>
+        <geometry>
+          <mesh filename="package://aidin_hand2_description/meshes/right_aidin_hand2/collision/right_palm1_tactile_link.STL"/>
+        </geometry>
+      </collision>
+    </link>
+    <link name="${prefix}palm2_tactile_link">
       <inertial>
         <origin xyz="0.000649300878208026 0.000641439582478615 0.0169329552007083" rpy="0 0 0"/>
@@ -78,27 +78,27 @@
         <origin xyz="0 0 0" rpy="0 0 0"/>
         <geometry>
-          <mesh filename="package://aidin_hand2_description/meshes/right_aidin_hand2/visual/right_palm_tactile_bottom_link.STL"/>
-        </geometry>
-        <material name="">
-          <color rgba="0.274509803921569 0.274509803921569 0.274509803921569 1"/>
-        </material>
-      </visual>
-      <collision>
-        <origin xyz="0 0 0" rpy="0 0 0"/>
-        <geometry>
-          <mesh filename="package://aidin_hand2_description/meshes/right_aidin_hand2/collision/right_palm_tactile_bottom_link.STL"/>
-        </geometry>
-      </collision>
-    </link>
-    <joint name="${prefix}palm_tactile_top_joint" type="fixed">
+          <mesh filename="package://aidin_hand2_description/meshes/right_aidin_hand2/visual/right_palm2_tactile_link.STL"/>
+        </geometry>
+        <material name="">
+          <color rgba="0.274509803921569 0.274509803921569 0.274509803921569 1"/>
+        </material>
+      </visual>
+      <collision>
+        <origin xyz="0 0 0" rpy="0 0 0"/>
+        <geometry>
+          <mesh filename="package://aidin_hand2_description/meshes/right_aidin_hand2/collision/right_palm2_tactile_link.STL"/>
+        </geometry>
+      </collision>
+    </link>
+    <joint name="${prefix}palm1_tactile_joint" type="fixed">
       <origin xyz="0.0305 0 0.0669" rpy="0 0 0"/>
       <parent link="${prefix}hand_base_link"/>
-      <child link="${prefix}palm_tactile_top_link"/>
-      <axis xyz="0 0 0"/>
-    </joint>
-    <joint name="${prefix}palm_tactile_bottom_joint" type="fixed">
+      <child link="${prefix}palm1_tactile_link"/>
+      <axis xyz="0 0 0"/>
+    </joint>
+    <joint name="${prefix}palm2_tactile_joint" type="fixed">
       <origin xyz="0.0305 -0.0205 0.0289" rpy="0 0 0"/>
       <parent link="${prefix}hand_base_link"/>
-      <child link="${prefix}palm_tactile_bottom_link"/>
+      <child link="${prefix}palm2_tactile_link"/>
       <axis xyz="0 0 0"/>
     </joint>

File: viewer/model/left.urdf (robot description, URDF)
Before this commit: robot aidin_hand2_left, 39 links, 38 joints
Links:
- removed link left_palm_tactile_bottom_link
- removed link left_palm_tactile_top_link
- added link left_palm1_tactile_link; visual mesh filename=package://viewer_model/meshes/visual/left_palm1_tactile_lin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
- added link left_palm2_tactile_link; visual mesh filename=package://viewer_model/meshes/visual/left_palm2_tactile_lin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
Joints:
- removed joint left_palm_tactile_bottom_joint
- removed joint left_palm_tactile_top_joint
- added joint left_palm1_tactile_joint: type fixed, parent left_hand_base_link, child left_palm1_tactile_link, origin xyz=0.0305 0 0.0669 rpy=0 0 0, axis 0 0 0
- added joint left_palm2_tactile_joint: type fixed, parent left_hand_base_link, child left_palm2_tactile_link, origin xyz=0.0305 0.0205 0.0289 rpy=0 0 0, axis 0 0 0

File: viewer/model/right.urdf (robot description, URDF)
Before this commit: robot aidin_hand2_right, 39 links, 38 joints
Links:
- removed link right_palm_tactile_bottom_link
- removed link right_palm_tactile_top_link
- added link right_palm1_tactile_link; visual mesh filename=package://viewer_model/meshes/visual/right_palm1_tactile_li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
- added link right_palm2_tactile_link; visual mesh filename=package://viewer_model/meshes/visual/right_palm2_tactile_li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
Joints:
- removed joint right_palm_tactile_bottom_joint
- removed joint right_palm_tactile_top_joint
- added joint right_palm1_tactile_joint: type fixed, parent right_hand_base_link, child right_palm1_tactile_link, origin xyz=0.0305 0 0.0669 rpy=0 0 0, axis 0 0 0
- added joint right_palm2_tactile_joint: type fixed, parent right_hand_base_link, child right_palm2_tactile_link, origin xyz=0.0305 -0.0205 0.0289 rpy=0 0 0, axis 0 0 0
