Commit message: fix(description): Match the remeasured workspace
The SDK clamp moved to the workspace measured after the mechanical
design change. The joint limits and the viewer's tables follow it.

File: aidin_hand2_description/urdf/aidin_hand2_left.urdf (robot description, URDF)
Before this commit: robot aidin_hand2_left, 39 links, 38 joints
Joints:
- joint left_baby_joint1: limit lower=-0.479966 upper=0.479966 effort=1.2 velocity=1.57 -> lower=-0.541052 upper=0.541052 effort=1.2 velocity=1.57
- joint left_baby_joint2: limit lower=0 upper=1.666091 effort=1.2 velocity=1.57 -> lower=0 upper=1.679007 effort=1.2 velocity=1.57
- joint left_baby_joint3: limit lower=0 upper=1.570796 effort=1.2 velocity=1.57 -> lower=0 upper=1.396263 effort=1.2 velocity=1.57
- joint left_baby_joint4: limit lower=0 upper=1.736252 effort=1.2 velocity=1.57 -> lower=0 upper=1.581268 effort=1.2 velocity=1.57
- joint left_index_joint1: limit lower=-0.479966 upper=0.479966 effort=1.2 velocity=1.57 -> lower=-0.541052 upper=0.541052 effort=1.2 velocity=1.57
- joint left_index_joint2: limit lower=0 upper=1.666091 effort=1.2 velocity=1.57 -> lower=0 upper=1.679007 effort=1.2 velocity=1.57
- joint left_index_joint3: limit lower=0 upper=1.570796 effort=1.2 velocity=1.57 -> lower=0 upper=1.396263 effort=1.2 velocity=1.57
- joint left_index_joint4: limit lower=0 upper=1.736252 effort=1.2 velocity=1.57 -> lower=0 upper=1.581268 effort=1.2 velocity=1.57
- joint left_middle_joint1: limit lower=-0.479966 upper=0.479966 effort=1.2 velocity=1.57 -> lower=-0.541052 upper=0.541052 effort=1.2 velocity=1.57
- joint left_middle_joint2: limit lower=0 upper=1.666091 effort=1.2 velocity=1.57 -> lower=0 upper=1.679007 effort=1.2 velocity=1.57
- joint left_middle_joint3: limit lower=0 upper=1.570796 effort=1.2 velocity=1.57 -> lower=0 upper=1.396263 effort=1.2 velocity=1.57
- joint left_middle_joint4: limit lower=0 upper=1.736252 effort=1.2 velocity=1.57 -> lower=0 upper=1.581268 effort=1.2 velocity=1.57
- joint left_ring_joint1: limit lower=-0.479966 upper=0.479966 effort=1.2 velocity=1.57 -> lower=-0.541052 upper=0.541052 effort=1.2 velocity=1.57
- joint left_ring_joint2: limit lower=0 upper=1.666091 effort=1.2 velocity=1.57 -> lower=0 upper=1.679007 effort=1.2 velocity=1.57
- joint left_ring_joint3: limit lower=0 upper=1.570796 effort=1.2 velocity=1.57 -> lower=0 upper=1.396263 effort=1.2 velocity=1.57
- joint left_ring_joint4: limit lower=0 upper=1.736252 effort=1.2 velocity=1.57 -> lower=0 upper=1.581268 effort=1.2 velocity=1.57
- joint left_thumb_joint0: limit lower=0 upper=1.919862 effort=1.2 velocity=1.57 -> lower=0 upper=1.898918 effort=1.2 velocity=1.57
- joint left_thumb_joint1: limit lower=0 upper=1.330464 effort=1.2 velocity=1.57 -> lower=0 upper=1.029744 effort=1.2 velocity=1.57
- joint left_thumb_joint2: limit lower=-0.787143 upper=0.787143 effort=1.2 velocity=1.57 -> lower=-0.776672 upper=0.776672 effort=1.2 velocity=1.57
- joint left_thumb_joint3: limit lower=0 upper=1.22173 effort=1.2 velocity=1.57 -> lower=0 upper=1.308997 effort=1.2 velocity=1.57
- joint left_thumb_joint4: limit lower=0 upper=1.316145 effort=1.2 velocity=1.57 -> lower=0 upper=1.480039 effort=1.2 velocity=1.57

File: aidin_hand2_description/urdf/aidin_hand2_right.urdf (robot description, URDF)
Before this commit: robot aidin_hand2_right, 39 links, 38 joints
Joints:
- joint right_baby_joint1: limit lower=-0.479966 upper=0.479966 effort=1.2 velocity=1.57 -> lower=-0.541052 upper=0.541052 effort=1.2 velocity=1.57
- joint right_baby_joint2: limit lower=0 upper=1.666091 effort=1.2 velocity=1.57 -> lower=0 upper=1.679007 effort=1.2 velocity=1.57
- joint right_baby_joint3: limit lower=0 upper=1.570796 effort=1.2 velocity=1.57 -> lower=0 upper=1.396263 effort=1.2 velocity=1.57
- joint right_baby_joint4: limit lower=0 upper=1.736252 effort=1.2 velocity=1.57 -> lower=0 upper=1.581268 effort=1.2 velocity=1.57
- joint right_index_joint1: limit lower=-0.479966 upper=0.479966 effort=1.2 velocity=1.57 -> lower=-0.541052 upper=0.541052 effort=1.2 velocity=1.57
- joint right_index_joint2: limit lower=0 upper=1.666091 effort=1.2 velocity=1.57 -> lower=0 upper=1.679007 effort=1.2 velocity=1.57
- joint right_index_joint3: limit lower=0 upper=1.570796 effort=1.2 velocity=1.57 -> lower=0 upper=1.396263 effort=1.2 velocity=1.57
- joint right_index_joint4: limit lower=0 upper=1.736252 effort=1.2 velocity=1.57 -> lower=0 upper=1.581268 effort=1.2 velocity=1.57
- joint right_middle_joint1: limit lower=-0.479966 upper=0.479966 effort=1.2 velocity=1.57 -> lower=-0.541052 upper=0.541052 effort=1.2 velocity=1.57
- joint right_middle_joint2: limit lower=0 upper=1.666091 effort=1.2 velocity=1.57 -> lower=0 upper=1.679007 effort=1.2 velocity=1.57
- joint right_middle_joint3: limit lower=0 upper=1.570796 effort=1.2 velocity=1.57 -> lower=0 upper=1.396263 effort=1.2 velocity=1.57
- joint right_middle_joint4: limit lower=0 upper=1.736252 effort=1.2 velocity=1.57 -> lower=0 upper=1.581268 effort=1.2 velocity=1.57
- joint right_ring_joint1: limit lower=-0.479966 upper=0.479966 effort=1.2 velocity=1.57 -> lower=-0.541052 upper=0.541052 effort=1.2 velocity=1.57
- joint right_ring_joint2: limit lower=0 upper=1.666091 effort=1.2 velocity=1.57 -> lower=0 upper=1.679007 effort=1.2 velocity=1.57
- joint right_ring_joint3: limit lower=0 upper=1.570796 effort=1.2 velocity=1.57 -> lower=0 upper=1.396263 effort=1.2 velocity=1.57
- joint right_ring_joint4: limit lower=0 upper=1.736252 effort=1.2 velocity=1.57 -> lower=0 upper=1.581268 effort=1.2 velocity=1.57
- joint right_thumb_joint0: limit lower=0 upper=1.919862 effort=1.2 velocity=1.57 -> lower=0 upper=1.898918 effort=1.2 velocity=1.57
- joint right_thumb_joint1: limit lower=0 upper=1.330464 effort=1.2 velocity=1.57 -> lower=0 upper=1.029744 effort=1.2 velocity=1.57
- joint right_thumb_joint2: limit lower=-0.787143 upper=0.787143 effort=1.2 velocity=1.57 -> lower=-0.776672 upper=0.776672 effort=1.2 velocity=1.57
- joint right_thumb_joint3: limit lower=0 upper=1.22173 effort=1.2 velocity=1.57 -> lower=0 upper=1.308997 effort=1.2 velocity=1.57
- joint right_thumb_joint4: limit lower=0 upper=1.316145 effort=1.2 velocity=1.57 -> lower=0 upper=1.480039 effort=1.2 velocity=1.57

File: aidin_hand2_description/xacro/aidin_hand2_left.urdf.xacro (robot description, xacro)
@@ -309,5 +309,5 @@
       <child link="${prefix}thumb_link0"/>
       <axis xyz="0 1 0"/>
-      <limit lower="0" upper="1.919862" effort="1.2" velocity="1.57"/>
+      <limit lower="0" upper="1.898918" effort="1.2" velocity="1.57"/>
     </joint>
     <joint name="${prefix}thumb_joint1" type="revolute">
@@ -316,5 +316,5 @@
       <child link="${prefix}thumb_link1"/>
       <axis xyz="0 1 0"/>
-      <limit lower="0" upper="1.330464" effort="1.2" velocity="1.57"/>
+      <limit lower="0" upper="1.029744" effort="1.2" velocity="1.57"/>
     </joint>
     <joint name="${prefix}thumb_joint2" type="revolute">
@@ -323,5 +323,5 @@
       <child link="${prefix}thumb_link2"/>
       <axis xyz="0 1 0"/>
-      <limit lower="-0.787143" upper="0.787143" effort="1.2" velocity="1.57"/>
+      <limit lower="-0.776672" upper="0.776672" effort="1.2" velocity="1.57"/>
     </joint>
     <joint name="${prefix}thumb_joint3" type="revolute">
@@ -330,5 +330,5 @@
       <child link="${prefix}thumb_link3"/>
       <axis xyz="0 1 0"/>
-      <limit lower="0" upper="1.22173" effort="1.2" velocity="1.57"/>
+      <limit lower="0" upper="1.308997" effort="1.2" velocity="1.57"/>
     </joint>
     <joint name="${prefix}thumb_joint4" type="revolute">
@@ -337,5 +337,5 @@
       <child link="${prefix}thumb_link4"/>
       <axis xyz="0 1 0"/>
-      <limit lower="0" upper="1.316145" effort="1.2" velocity="1.57"/>
+      <limit lower="0" upper="1.480039" effort="1.2" velocity="1.57"/>
     </joint>
     <joint name="${prefix}thumb_tactile_joint2" type="fixed">
@@ -538,5 +538,5 @@
       <child link="${prefix}index_link1"/>
       <axis xyz="0 1 0"/>
-      <limit lower="-0.479966" upper="0.479966" effort="1.2" velocity="1.57"/>
+      <limit lower="-0.541052" upper="0.541052" effort="1.2" velocity="1.57"/>
     </joint>
     <joint name="${prefix}index_joint2" type="revolute">
@@ -545,5 +545,5 @@
       <child link="${prefix}index_link2"/>
       <axis xyz="0 1 0"/>
-      <limit lower="0" upper="1.666091" effort="1.2" velocity="1.57"/>
+      <limit lower="0" upper="1.679007" effort="1.2" velocity="1.57"/>
     </joint>
     <joint name="${prefix}index_joint3" type="revolute">
@@ -552,5 +552,5 @@
       <child link="${prefix}index_link3"/>
       <axis xyz="0 1 0"/>
-      <limit lower="0" upper="1.570796" effort="1.2" velocity="1.57"/>
+      <limit lower="0" upper="1.396263" effort="1.2" velocity="1.57"/>
     </joint>
     <joint name="${prefix}index_joint4" type="revolute">
@@ -559,5 +559,5 @@
       <child link="${prefix}index_link4"/>
       <axis xyz="0 1 0"/>
-      <limit lower="0" upper="1.736252" effort="1.2" velocity="1.57"/>
+      <limit lower="0" upper="1.581268" effort="1.2" velocity="1.57"/>
     </joint>
     <joint name="${prefix}index_tactile_joint2" type="fixed">
@@ -760,5 +760,5 @@
       <child link="${prefix}middle_link1"/>
       <axis xyz="0 1 0"/>
-      <limit lower="-0.479966" upper="0.479966" effort="1.2" velocity="1.57"/>
+      <limit lower="-0.541052" upper="0.541052" effort="1.2" velocity="1.57"/>
     </joint>
     <joint name="${prefix}middle_joint2" type="revolute">
@@ -767,5 +767,5 @@
       <child link="${prefix}middle_link2"/>
       <axis xyz="0 1 0"/>
-      <limit lower="0" upper="1.666091" effort="1.2" velocity="1.57"/>
+      <limit lower="0" upper="1.679007" effort="1.2" velocity="1.57"/>
     </joint>
     <joint name="${prefix}middle_joint3" type="revolute">
@@ -774,5 +774,5 @@
       <child link="${prefix}middle_link3"/>
       <axis xyz="0 1 0"/>
-      <limit lower="0" upper="1.570796" effort="1.2" velocity="1.57"/>
+      <limit lower="0" upper="1.396263" effort="1.2" velocity="1.57"/>
     </joint>
     <joint name="${prefix}middle_joint4" type="revolute">
@@ -781,5 +781,5 @@
       <child link="${prefix}middle_link4"/>
       <axis xyz="0 1 0"/>
-      <limit lower="0" upper="1.736252" effort="1.2" velocity="1.57"/>
+      <limit lower="0" upper="1.581268" effort="1.2" velocity="1.57"/>
     </joint>
     <joint name="${prefix}middle_tactile_joint2" type="fixed">
@@ -982,5 +982,5 @@
       <child link="${prefix}ring_link1"/>
       <axis xyz="0 1 0"/>
-      <limit lower="-0.479966" upper="0.479966" effort="1.2" velocity="1.57"/>
+      <limit lower="-0.541052" upper="0.541052" effort="1.2" velocity="1.57"/>
     </joint>
     <joint name="${prefix}ring_joint2" type="revolute">
@@ -989,5 +989,5 @@
       <child link="${prefix}ring_link2"/>
       <axis xyz="0 1 0"/>
-      <limit lower="0" upper="1.666091" effort="1.2" velocity="1.57"/>
+      <limit lower="0" upper="1.679007" effort="1.2" velocity="1.57"/>
     </joint>
     <joint name="${prefix}ring_joint3" type="revolute">
@@ -996,5 +996,5 @@
       <child link="${prefix}ring_link3"/>
       <axis xyz="0 1 0"/>
-      <limit lower="0" upper="1.570796" effort="1.2" velocity="1.57"/>
+      <limit lower="0" upper="1.396263" effort="1.2" velocity="1.57"/>
     </joint>
     <joint name="${prefix}ring_joint4" type="revolute">
@@ -1003,5 +1003,5 @@
       <child link="${prefix}ring_link4"/>
       <axis xyz="0 1 0"/>
-      <limit lower="0" upper="1.736252" effort="1.2" velocity="1.57"/>
+      <limit lower="0" upper="1.581268" effort="1.2" velocity="1.57"/>
     </joint>
     <joint name="${prefix}ring_tactile_joint2" type="fixed">
@@ -1204,5 +1204,5 @@
       <child link="${prefix}baby_link1"/>
       <axis xyz="0 1 0"/>
-      <limit lower="-0.479966" upper="0.479966" effort="1.2" velocity="1.57"/>
+      <limit lower="-0.541052" upper="0.541052" effort="1.2" velocity="1.57"/>
     </joint>
     <joint name="${prefix}baby_joint2" type="revolute">
@@ -1211,5 +1211,5 @@
       <child link="${prefix}baby_link2"/>
       <axis xyz="0 1 0"/>
-      <limit lower="0" upper="1.666091" effort="1.2" velocity="1.57"/>
+      <limit lower="0" upper="1.679007" effort="1.2" velocity="1.57"/>
     </joint>
     <joint name="${prefix}baby_joint3" type="revolute">
@@ -1218,5 +1218,5 @@
       <child link="${prefix}baby_link3"/>
       <axis xyz="0 1 0"/>
-      <limit lower="0" upper="1.570796" effort="1.2" velocity="1.57"/>
+      <limit lower="0" upper="1.396263" effort="1.2" velocity="1.57"/>
     </joint>
     <joint name="${prefix}baby_joint4" type="revolute">
@@ -1225,5 +1225,5 @@
       <child link="${prefix}baby_link4"/>
       <axis xyz="0 1 0"/>
-      <limit lower="0" upper="1.736252" effort="1.2" velocity="1.57"/>
+      <limit lower="0" upper="1.581268" effort="1.2" velocity="1.57"/>
     </joint>
     <joint name="${prefix}baby_tactile_joint2" type="fixed">

File: aidin_hand2_description/xacro/aidin_hand2_right.urdf.xacro (robot description, xacro)
@@ -309,5 +309,5 @@
       <child link="${prefix}thumb_link0"/>
       <axis xyz="0 1 0"/>
-      <limit lower="0" upper="1.919862" effort="1.2" velocity="1.57"/>
+      <limit lower="0" upper="1.898918" effort="1.2" velocity="1.57"/>
     </joint>
     <joint name="${prefix}thumb_joint1" type="revolute">
@@ -316,5 +316,5 @@
       <child link="${prefix}thumb_link1"/>
       <axis xyz="0 1 0"/>
-      <limit lower="0" upper="1.330464" effort="1.2" velocity="1.57"/>
+      <limit lower="0" upper="1.029744" effort="1.2" velocity="1.57"/>
     </joint>
     <joint name="${prefix}thumb_joint2" type="revolute">
@@ -323,5 +323,5 @@
       <child link="${prefix}thumb_link2"/>
       <axis xyz="0 1 0"/>
-      <limit lower="-0.787143" upper="0.787143" effort="1.2" velocity="1.57"/>
+      <limit lower="-0.776672" upper="0.776672" effort="1.2" velocity="1.57"/>
     </joint>
     <joint name="${prefix}thumb_joint3" type="revolute">
@@ -330,5 +330,5 @@
       <child link="${prefix}thumb_link3"/>
       <axis xyz="0 1 0"/>
-      <limit lower="0" upper="1.22173" effort="1.2" velocity="1.57"/>
+      <limit lower="0" upper="1.308997" effort="1.2" velocity="1.57"/>
     </joint>
     <joint name="${prefix}thumb_joint4" type="revolute">
@@ -337,5 +337,5 @@
       <child link="${prefix}thumb_link4"/>
       <axis xyz="0 1 0"/>
-      <limit lower="0" upper="1.316145" effort="1.2" velocity="1.57"/>
+      <limit lower="0" upper="1.480039" effort="1.2" velocity="1.57"/>
     </joint>
     <joint name="${prefix}thumb_tactile_joint2" type="fixed">
@@ -538,5 +538,5 @@
       <child link="${prefix}index_link1"/>
       <axis xyz="0 1 0"/>
-      <limit lower="-0.479966" upper="0.479966" effort="1.2" velocity="1.57"/>
+      <limit lower="-0.541052" upper="0.541052" effort="1.2" velocity="1.57"/>
     </joint>
     <joint name="${prefix}index_joint2" type="revolute">
@@ -545,5 +545,5 @@
       <child link="${prefix}index_link2"/>
       <axis xyz="0 1 0"/>
-      <limit lower="0" upper="1.666091" effort="1.2" velocity="1.57"/>
+      <limit lower="0" upper="1.679007" effort="1.2" velocity="1.57"/>
     </joint>
     <joint name="${prefix}index_joint3" type="revolute">
@@ -552,5 +552,5 @@
       <child link="${prefix}index_link3"/>
       <axis xyz="0 1 0"/>
-      <limit lower="0" upper="1.570796" effort="1.2" velocity="1.57"/>
+      <limit lower="0" upper="1.396263" effort="1.2" velocity="1.57"/>
     </joint>
     <joint name="${prefix}index_joint4" type="revolute">
@@ -559,5 +559,5 @@
       <child link="${prefix}index_link4"/>
       <axis xyz="0 1 0"/>
-      <limit lower="0" upper="1.736252" effort="1.2" velocity="1.57"/>
+      <limit lower="0" upper="1.581268" effort="1.2" velocity="1.57"/>
     </joint>
     <joint name="${prefix}index_tactile_joint2" type="fixed">
@@ -760,5 +760,5 @@
       <child link="${prefix}middle_link1"/>
       <axis xyz="0 1 0"/>
-      <limit lower="-0.479966" upper="0.479966" effort="1.2" velocity="1.57"/>
+      <limit lower="-0.541052" upper="0.541052" effort="1.2" velocity="1.57"/>
     </joint>
     <joint name="${prefix}middle_joint2" type="revolute">
@@ -767,5 +767,5 @@
       <child link="${prefix}middle_link2"/>
       <axis xyz="0 1 0"/>
-      <limit lower="0" upper="1.666091" effort="1.2" velocity="1.57"/>
+      <limit lower="0" upper="1.679007" effort="1.2" velocity="1.57"/>
     </joint>
     <joint name="${prefix}middle_joint3" type="revolute">
@@ -774,5 +774,5 @@
       <child link="${prefix}middle_link3"/>
       <axis xyz="0 1 0"/>
-      <limit lower="0" upper="1.570796" effort="1.2" velocity="1.57"/>
+      <limit lower="0" upper="1.396263" effort="1.2" velocity="1.57"/>
     </joint>
     <joint name="${prefix}middle_joint4" type="revolute">
@@ -781,5 +781,5 @@
       <child link="${prefix}middle_link4"/>
       <axis xyz="0 1 0"/>
-      <limit lower="0" upper="1.736252" effort="1.2" velocity="1.57"/>
+      <limit lower="0" upper="1.581268" effort="1.2" velocity="1.57"/>
     </joint>
     <joint name="${prefix}middle_tactile_joint2" type="fixed">
@@ -982,5 +982,5 @@
       <child link="${prefix}ring_link1"/>
       <axis xyz="0 1 0"/>
-      <limit lower="-0.479966" upper="0.479966" effort="1.2" velocity="1.57"/>
+      <limit lower="-0.541052" upper="0.541052" effort="1.2" velocity="1.57"/>
     </joint>
     <joint name="${prefix}ring_joint2" type="revolute">
@@ -989,5 +989,5 @@
       <child link="${prefix}ring_link2"/>
       <axis xyz="0 1 0"/>
-      <limit lower="0" upper="1.666091" effort="1.2" velocity="1.57"/>
+      <limit lower="0" upper="1.679007" effort="1.2" velocity="1.57"/>
     </joint>
     <joint name="${prefix}ring_joint3" type="revolute">
@@ -996,5 +996,5 @@
       <child link="${prefix}ring_link3"/>
       <axis xyz="0 1 0"/>
-      <limit lower="0" upper="1.570796" effort="1.2" velocity="1.57"/>
+      <limit lower="0" upper="1.396263" effort="1.2" velocity="1.57"/>
     </joint>
     <joint name="${prefix}ring_joint4" type="revolute">
@@ -1003,5 +1003,5 @@
       <child link="${prefix}ring_link4"/>
       <axis xyz="0 1 0"/>
-      <limit lower="0" upper="1.736252" effort="1.2" velocity="1.57"/>
+      <limit lower="0" upper="1.581268" effort="1.2" velocity="1.57"/>
     </joint>
     <joint name="${prefix}ring_tactile_joint2" type="fixed">
@@ -1204,5 +1204,5 @@
       <child link="${prefix}baby_link1"/>
       <axis xyz="0 1 0"/>
-      <limit lower="-0.479966" upper="0.479966" effort="1.2" velocity="1.57"/>
+      <limit lower="-0.541052" upper="0.541052" effort="1.2" velocity="1.57"/>
     </joint>
     <joint name="${prefix}baby_joint2" type="revolute">
@@ -1211,5 +1211,5 @@
       <child link="${prefix}baby_link2"/>
       <axis xyz="0 1 0"/>
-      <limit lower="0" upper="1.666091" effort="1.2" velocity="1.57"/>
+      <limit lower="0" upper="1.679007" effort="1.2" velocity="1.57"/>
     </joint>
     <joint name="${prefix}baby_joint3" type="revolute">
@@ -1218,5 +1218,5 @@
       <child link="${prefix}baby_link3"/>
       <axis xyz="0 1 0"/>
-      <limit lower="0" upper="1.570796" effort="1.2" velocity="1.57"/>
+      <limit lower="0" upper="1.396263" effort="1.2" velocity="1.57"/>
     </joint>
     <joint name="${prefix}baby_joint4" type="revolute">
@@ -1225,5 +1225,5 @@
       <child link="${prefix}baby_link4"/>
       <axis xyz="0 1 0"/>
-      <limit lower="0" upper="1.736252" effort="1.2" velocity="1.57"/>
+      <limit lower="0" upper="1.581268" effort="1.2" velocity="1.57"/>
     </joint>
     <joint name="${prefix}baby_tactile_joint2" type="fixed">

File: viewer/model/left.urdf (robot description, URDF)
Before this commit: robot aidin_hand2_left, 39 links, 38 joints
Joints:
- joint left_baby_joint1: limit lower=-0.479966 upper=0.479966 effort=1.2 velocity=1.57 -> lower=-0.541052 upper=0.541052 effort=1.2 velocity=1.57
- joint left_baby_joint2: limit lower=0 upper=1.666091 effort=1.2 velocity=1.57 -> lower=0 upper=1.679007 effort=1.2 velocity=1.57
- joint left_baby_joint3: limit lower=0 upper=1.570796 effort=1.2 velocity=1.57 -> lower=0 upper=1.396263 effort=1.2 velocity=1.57
- joint left_baby_joint4: limit lower=0 upper=1.736252 effort=1.2 velocity=1.57 -> lower=0 upper=1.581268 effort=1.2 velocity=1.57
- joint left_index_joint1: limit lower=-0.479966 upper=0.479966 effort=1.2 velocity=1.57 -> lower=-0.541052 upper=0.541052 effort=1.2 velocity=1.57
- joint left_index_joint2: limit lower=0 upper=1.666091 effort=1.2 velocity=1.57 -> lower=0 upper=1.679007 effort=1.2 velocity=1.57
- joint left_index_joint3: limit lower=0 upper=1.570796 effort=1.2 velocity=1.57 -> lower=0 upper=1.396263 effort=1.2 velocity=1.57
- joint left_index_joint4: limit lower=0 upper=1.736252 effort=1.2 velocity=1.57 -> lower=0 upper=1.581268 effort=1.2 velocity=1.57
- joint left_middle_joint1: limit lower=-0.479966 upper=0.479966 effort=1.2 velocity=1.57 -> lower=-0.541052 upper=0.541052 effort=1.2 velocity=1.57
- joint left_middle_joint2: limit lower=0 upper=1.666091 effort=1.2 velocity=1.57 -> lower=0 upper=1.679007 effort=1.2 velocity=1.57
- joint left_middle_joint3: limit lower=0 upper=1.570796 effort=1.2 velocity=1.57 -> lower=0 upper=1.396263 effort=1.2 velocity=1.57
- joint left_middle_joint4: limit lower=0 upper=1.736252 effort=1.2 velocity=1.57 -> lower=0 upper=1.581268 effort=1.2 velocity=1.57
- joint left_ring_joint1: limit lower=-0.479966 upper=0.479966 effort=1.2 velocity=1.57 -> lower=-0.541052 upper=0.541052 effort=1.2 velocity=1.57
- joint left_ring_joint2: limit lower=0 upper=1.666091 effort=1.2 velocity=1.57 -> lower=0 upper=1.679007 effort=1.2 velocity=1.57
- joint left_ring_joint3: limit lower=0 upper=1.570796 effort=1.2 velocity=1.57 -> lower=0 upper=1.396263 effort=1.2 velocity=1.57
- joint left_ring_joint4: limit lower=0 upper=1.736252 effort=1.2 velocity=1.57 -> lower=0 upper=1.581268 effort=1.2 velocity=1.57
- joint left_thumb_joint0: limit lower=0 upper=1.919862 effort=1.2 velocity=1.57 -> lower=0 upper=1.898918 effort=1.2 velocity=1.57
- joint left_thumb_joint1: limit lower=0 upper=1.330464 effort=1.2 velocity=1.57 -> lower=0 upper=1.029744 effort=1.2 velocity=1.57
- joint left_thumb_joint2: limit lower=-0.787143 upper=0.787143 effort=1.2 velocity=1.57 -> lower=-0.776672 upper=0.776672 effort=1.2 velocity=1.57
- joint left_thumb_joint3: limit lower=0 upper=1.22173 effort=1.2 velocity=1.57 -> lower=0 upper=1.308997 effort=1.2 velocity=1.57
- joint left_thumb_joint4: limit lower=0 upper=1.316145 effort=1.2 velocity=1.57 -> lower=0 upper=1.480039 effort=1.2 velocity=1.57
