Commit message: fix(viewer): Regenerate the model for the SDK joint bounds
The joint limits moved in the xacro without a rerun of
viewer/build-model, so the Pages check failed on main.

File: viewer/model/left.urdf (robot description, URDF)
Before this commit: robot aidin_hand2_left, 39 links, 38 joints
Joints:
- joint left_baby_joint1: limit lower=-0.5236 upper=0.5236 effort=1.2 velocity=1.57 -> lower=-0.479966 upper=0.479966 effort=1.2 velocity=1.57
- joint left_baby_joint2: limit lower=0 upper=1.6581 effort=1.2 velocity=1.57 -> lower=0 upper=1.666091 effort=1.2 velocity=1.57
- joint left_baby_joint3: limit lower=0 upper=1.5533 effort=1.2 velocity=1.57 -> lower=0 upper=1.570796 effort=1.2 velocity=1.57
- joint left_baby_joint4: limit lower=0 upper=1.6319 effort=1.2 velocity=1.57 -> lower=0 upper=1.736252 effort=1.2 velocity=1.57
- joint left_index_joint1: limit lower=-0.5236 upper=0.5236 effort=1.2 velocity=1.57 -> lower=-0.479966 upper=0.479966 effort=1.2 velocity=1.57
- joint left_index_joint2: limit lower=0 upper=1.6581 effort=1.2 velocity=1.57 -> lower=0 upper=1.666091 effort=1.2 velocity=1.57
- joint left_index_joint3: limit lower=0 upper=1.5533 effort=1.2 velocity=1.57 -> lower=0 upper=1.570796 effort=1.2 velocity=1.57
- joint left_index_joint4: limit lower=0 upper=1.6319 effort=1.2 velocity=1.57 -> lower=0 upper=1.736252 effort=1.2 velocity=1.57
- joint left_middle_joint1: limit lower=-0.5236 upper=0.5236 effort=1.2 velocity=1.57 -> lower=-0.479966 upper=0.479966 effort=1.2 velocity=1.57
- joint left_middle_joint2: limit lower=0 upper=1.6581 effort=1.2 velocity=1.57 -> lower=0 upper=1.666091 effort=1.2 velocity=1.57
- joint left_middle_joint3: limit lower=0 upper=1.5533 effort=1.2 velocity=1.57 -> lower=0 upper=1.570796 effort=1.2 velocity=1.57
- joint left_middle_joint4: limit lower=0 upper=1.6319 effort=1.2 velocity=1.57 -> lower=0 upper=1.736252 effort=1.2 velocity=1.57
- joint left_ring_joint1: limit lower=-0.5236 upper=0.5236 effort=1.2 velocity=1.57 -> lower=-0.479966 upper=0.479966 effort=1.2 velocity=1.57
- joint left_ring_joint2: limit lower=0 upper=1.6581 effort=1.2 velocity=1.57 -> lower=0 upper=1.666091 effort=1.2 velocity=1.57
- joint left_ring_joint3: limit lower=0 upper=1.5533 effort=1.2 velocity=1.57 -> lower=0 upper=1.570796 effort=1.2 velocity=1.57
- joint left_ring_joint4: limit lower=0 upper=1.6319 effort=1.2 velocity=1.57 -> lower=0 upper=1.736252 effort=1.2 velocity=1.57
- joint left_thumb_joint0: limit lower=0 upper=1.9084 effort=1.2 velocity=1.57 -> lower=0 upper=1.919862 effort=1.2 velocity=1.57
- joint left_thumb_joint1: limit lower=0 upper=1.2645 effort=1.2 velocity=1.57 -> lower=0 upper=1.330464 effort=1.2 velocity=1.57
- joint left_thumb_joint2: limit lower=-0.63668 upper=0.63668 effort=1.2 velocity=1.57 -> lower=-0.787143 upper=0.787143 effort=1.2 velocity=1.57
- joint left_thumb_joint3: limit lower=0 upper=1.1019 effort=1.2 velocity=1.57 -> lower=0 upper=1.22173 effort=1.2 velocity=1.57
- joint left_thumb_joint4: limit lower=0 upper=1.4479 effort=1.2 velocity=1.57 -> lower=0 upper=1.316145 effort=1.2 velocity=1.57

File: viewer/model/right.urdf (robot description, URDF)
Before this commit: robot aidin_hand2_right, 39 links, 38 joints
Joints:
- joint right_baby_joint1: limit lower=-0.5236 upper=0.5236 effort=1.2 velocity=1.57 -> lower=-0.479966 upper=0.479966 effort=1.2 velocity=1.57
- joint right_baby_joint2: limit lower=0 upper=1.6581 effort=1.2 velocity=1.57 -> lower=0 upper=1.666091 effort=1.2 velocity=1.57
- joint right_baby_joint3: limit lower=0 upper=1.5533 effort=1.2 velocity=1.57 -> lower=0 upper=1.570796 effort=1.2 velocity=1.57
- joint right_baby_joint4: limit lower=0 upper=1.6319 effort=1.2 velocity=1.57 -> lower=0 upper=1.736252 effort=1.2 velocity=1.57
- joint right_index_joint1: limit lower=-0.5236 upper=0.5236 effort=1.2 velocity=1.57 -> lower=-0.479966 upper=0.479966 effort=1.2 velocity=1.57
- joint right_index_joint2: limit lower=0 upper=1.6581 effort=1.2 velocity=1.57 -> lower=0 upper=1.666091 effort=1.2 velocity=1.57
- joint right_index_joint3: limit lower=0 upper=1.5533 effort=1.2 velocity=1.57 -> lower=0 upper=1.570796 effort=1.2 velocity=1.57
- joint right_index_joint4: limit lower=0 upper=1.6319 effort=1.2 velocity=1.57 -> lower=0 upper=1.736252 effort=1.2 velocity=1.57
- joint right_middle_joint1: limit lower=-0.5236 upper=0.5236 effort=1.2 velocity=1.57 -> lower=-0.479966 upper=0.479966 effort=1.2 velocity=1.57
- joint right_middle_joint2: limit lower=0 upper=1.6581 effort=1.2 velocity=1.57 -> lower=0 upper=1.666091 effort=1.2 velocity=1.57
- joint right_middle_joint3: limit lower=0 upper=1.5533 effort=1.2 velocity=1.57 -> lower=0 upper=1.570796 effort=1.2 velocity=1.57
- joint right_middle_joint4: limit lower=0 upper=1.6319 effort=1.2 velocity=1.57 -> lower=0 upper=1.736252 effort=1.2 velocity=1.57
- joint right_ring_joint1: limit lower=-0.5236 upper=0.5236 effort=1.2 velocity=1.57 -> lower=-0.479966 upper=0.479966 effort=1.2 velocity=1.57
- joint right_ring_joint2: limit lower=0 upper=1.6581 effort=1.2 velocity=1.57 -> lower=0 upper=1.666091 effort=1.2 velocity=1.57
- joint right_ring_joint3: limit lower=0 upper=1.5533 effort=1.2 velocity=1.57 -> lower=0 upper=1.570796 effort=1.2 velocity=1.57
- joint right_ring_joint4: limit lower=0 upper=1.6319 effort=1.2 velocity=1.57 -> lower=0 upper=1.736252 effort=1.2 velocity=1.57
- joint right_thumb_joint0: limit lower=0 upper=1.9084 effort=1.2 velocity=1.57 -> lower=0 upper=1.919862 effort=1.2 velocity=1.57
- joint right_thumb_joint1: limit lower=0 upper=1.2645 effort=1.2 velocity=1.57 -> lower=0 upper=1.330464 effort=1.2 velocity=1.57
- joint right_thumb_joint2: limit lower=-0.63668 upper=0.63668 effort=1.2 velocity=1.57 -> lower=-0.787143 upper=0.787143 effort=1.2 velocity=1.57
- joint right_thumb_joint3: limit lower=0 upper=1.1019 effort=1.2 velocity=1.57 -> lower=0 upper=1.22173 effort=1.2 velocity=1.57
- joint right_thumb_joint4: limit lower=0 upper=1.4479 effort=1.2 velocity=1.57 -> lower=0 upper=1.316145 effort=1.2 velocity=1.57
